Commit message: component_sorting_description: -Modified holder links for to update pick and place positions -Modified table base_link position

File: component_sorting_description/urdf/box/holder_robot.urdf.xacro (robot description, xacro)
@@ -30,23 +30,23 @@
         </geometry>
       </visual>
-      <collision>
+<!--       <collision>
         <origin rpy="0 0 0" xyz="0 0 0"/>
         <geometry>
           <mesh filename="package://component_sorting_description/meshes/box/box_holder.stl"/>
         </geometry>
-      </collision>
+      </collision>  -->
     </link>
-    <joint name="${prefix}approach_joint" type="fixed">
+    <joint name="${prefix}holder_approach_joint" type="fixed">
       <origin rpy="3.1416 0 0" xyz="-0.075 0 0.741"/>
       <parent link="${prefix}holder_link"/>
-      <child link="${prefix}approach"/>
+      <child link="${prefix}holder_approach"/>
     </joint>
-    <link name="${prefix}approach"/>
-    <joint name="${prefix}grab_joint" type="fixed">
+    <link name="${prefix}holder_approach"/>
+<!--     <joint name="${prefix}grab_joint" type="fixed">
       <origin rpy="3.1416 0 0" xyz="0.0 0 0.371"/>
       <parent link="${prefix}holder_link"/>
       <child link="${prefix}grab"/>
     </joint>
-    <link name="${prefix}grab"/>
+    <link name="${prefix}grab"/> -->
     <!-- TABLE TAG -->
     <xacro:ar_tag prefix="${prefix}" parent="${prefix}holder_link" tag_id="${tag_id}">

File: component_sorting_description/urdf/box/holder_table.urdf.xacro (robot description, xacro)
@@ -38,16 +38,16 @@
       </collision>
     </link>
-    <joint name="${prefix}approach_joint" type="fixed">
+    <joint name="${prefix}holder_approach_joint" type="fixed">
       <origin rpy="3.1416 0 0" xyz="-0.137 0 0.50"/>
       <parent link="${prefix}holder_link"/>
-      <child link="${prefix}approach"/>
+      <child link="${prefix}holder_approach"/>
     </joint>
-    <link name="${prefix}approach"/>
-    <joint name="${prefix}grab_joint" type="fixed">
+    <link name="${prefix}holder_approach"/>
+<!--     <joint name="${prefix}grab_joint" type="fixed">
       <origin rpy="3.1416 0 0" xyz="0 0 0.38"/>
       <parent link="${prefix}holder_link"/>
       <child link="${prefix}grab"/>
     </joint>
-    <link name="${prefix}grab"/>
+    <link name="${prefix}grab"/> -->
     <!-- TABLE TAG -->
     <xacro:ar_tag prefix="${prefix}holder_" parent="${prefix}holder_link" tag_id="${tag_id}">

File: component_sorting_description/urdf/table.urdf.xacro (robot description, xacro)
@@ -26,5 +26,5 @@
       <updateRate>50.0</updateRate>
       <bodyName>${prefix}qr</bodyName>
-      <frameName>${prefix}qr_tf</frameName>
+      <frameName>${prefix}qr_gt</frameName>
       <worldBodyName>world</worldBodyName>
       <worldFrameName>robot_map</worldFrameName>
@@ -40,5 +40,5 @@
   </link>
   <joint name="${prefix}base_joint" type="fixed">
-    <origin rpy="0 0 0" xyz="${table_length/2}  0 ${-qr_height}"/>
+    <origin rpy="0 0 0" xyz="${table_length/2}  0 ${-qr_height+table_height/2}"/>
     <parent link="${prefix}qr"/>
     <child link="${prefix}base_link"/>
@@ -47,9 +47,9 @@
     <inertial>
       <mass value="70" />
-      <origin xyz="0 0 ${table_height/2}" rpy="0 0 0" />
+      <origin xyz="0 0 0" rpy="0 0 0" />
       <solid_cuboid_inertia m="70" h="${table_height}" d="${table_length}" w="${table_width}"/>
     </inertial>
     <visual>
-      <origin xyz="0 0 ${table_height/2}"/>
+      <origin xyz="0 0 0"/>
       <geometry>
         <box size="${table_length} ${table_width} ${table_height}" />
@@ -57,5 +57,5 @@
     </visual>
     <collision>
-      <origin xyz="0 0 ${table_height/2}"/>
+      <origin xyz="0 0 0"/>
       <geometry>
         <box size="${table_length} ${table_width} ${table_height}" />
@@ -69,11 +69,11 @@
   <xacro:property name="center_holder_offset_x" value="${(holder_length-table_length)/2}"/>
   <xacro:property name="center_holder_offset_y" value="0.0"/>
-  <xacro:property name="center_holder_offset_z" value="${table_height}"/>
+  <xacro:property name="center_holder_offset_z" value="${table_height/2}"/>
   <xacro:property name="left_holder_offset_x" value="${(holder_length-table_length)/2}"/> <!-- -0.195 -->
   <xacro:property name="left_holder_offset_y" value="${holder_width}"/> <!-- 0.225 -->
-  <xacro:property name="left_holder_offset_z" value="${table_height}"/>
+  <xacro:property name="left_holder_offset_z" value="${table_height/2}"/>
   <xacro:property name="right_holder_offset_x" value="${(holder_length-table_length)/2}"/>
   <xacro:property name="right_holder_offset_y" value="${-holder_width}"/>
-  <xacro:property name="right_holder_offset_z" value="${table_height}"/>
+  <xacro:property name="right_holder_offset_z" value="${table_height/2}"/>
     <!-- HOLDERS -->
   <xacro:holder_table prefix="${prefix}center_" parent="${prefix}base_link" tag_id="marker2_12cm" >
