Commit message: component_sorting_description: modify table, box and holder urdf to adapt to new orientation in ar_tag urdf

File: component_sorting_description/urdf/box/box.urdf.xacro (robot description, xacro)
@@ -87,5 +87,5 @@
   <!-- AR TAG -->
   <xacro:ar_tag prefix="${prefix}" parent="${prefix}handle_link" tag_id="${tag_id}">
-    <origin xyz="0 0 0.1575" rpy="0 0 0"/>
+    <origin xyz="0 0 0.1575" rpy="0 0 ${-3.14159/2}"/>
   </xacro:ar_tag>
 <!--  <xacro:artag name="artag_01" parent="${prefix}grasping_link">

File: component_sorting_description/urdf/box/holder.urdf.xacro (robot description, xacro)
@@ -52,5 +52,5 @@
     <!-- TABLE TAG -->
     <xacro:ar_tag prefix="${prefix}holder_" parent="${prefix}holder_link" tag_id="${tag_id}">
-      <origin xyz="0 0 0" rpy="0 0 0"/>
+      <origin xyz="0 0 0" rpy="0 0 ${-3.14159/2}"/>
     </xacro:ar_tag>
     <gazebo reference="${prefix}holder_link">

File: component_sorting_description/urdf/table.urdf.xacro (robot description, xacro)
@@ -57,6 +57,6 @@
     </collision>
   </link>
-  <joint name="${prefix}base_joint" type="fixed">
-    <origin rpy="0 0 0" xyz="${-table_length/2}  0 ${+qr_height}"/>
+  <joint name="${prefix}qr_joint" type="fixed">
+    <origin rpy="${+3.14159/2} 0 ${-3.14159/2}" xyz="${-table_length/2}  0 ${+qr_height}"/>
     <parent link="${prefix}base_link"/>
     <child link="${prefix}qr"/>
@@ -64,7 +64,14 @@
   <link name="${prefix}qr">
   </link>
+  <joint name="${prefix}docking_joint" type="fixed">
+    <origin rpy="0 ${+3.14159/2} ${+3.14159/2}" xyz="0 0 0.115"/>
+    <parent link="${prefix}qr"/>
+    <child link="${prefix}docking"/>
+  </joint>
+  <link name="${prefix}docking">
+  </link>
         <!-- TABLE TAG -->
   <xacro:ar_tag prefix="${prefix}" parent="${prefix}qr" tag_id="marker10_12cm">
-      <origin xyz="0 0 0" rpy="0 ${-3.14159/2} 0"/>
+      <origin xyz="0 0 0" rpy="0 0 0"/>
   </xacro:ar_tag>
   <xacro:property name="center_holder_offset_x" value="${(holder_length-table_length)/2}"/>

Commit message: component_sorting_description: reduce hanlde box displacement (better performance in simulation)

File: component_sorting_description/urdf/box/box.urdf.xacro (robot description, xacro)
@@ -55,5 +55,5 @@
   <joint name="${prefix}handle_joint" type="prismatic">
     <axis xyz="0 0 1"/>
-    <limit effort="1000.0" lower="-0.025" upper="0.025" velocity="0.5"/>
+    <limit effort="1000.0" lower="-0.02" upper="0.02" velocity="0.5"/>
     <origin rpy="0 0 0" xyz="0 0 0.1"/>
     <parent link="${prefix}body_box_link"/>
