Commit message: component_sorting_description: remove ar tag in holder + add collision bumpers to avoid boxes moving in gazebo when placed on top of kairos

File: component_sorting_description/urdf/box/holder.urdf.xacro (robot description, xacro)
@@ -20,7 +20,7 @@
     <link name="${prefix}holder_link">
       <inertial>
-        <mass value="0.1" />
+        <mass value="0.01" />
         <origin xyz="0 0.011 0" />
-        <xacro:solid_cuboid_inertia m="0.1" h="0.022" d="0.225" w="0.31">
+        <xacro:solid_cuboid_inertia m="0.01" h="0.022" d="0.225" w="0.31">
         </xacro:solid_cuboid_inertia>
       </inertial>
@@ -58,7 +58,105 @@
     <link name="${prefix}grab_link"/>
     <!-- TABLE TAG -->
-    <xacro:ar_tag prefix="${prefix}holder_" parent="${prefix}holder_link" tag_id="${tag_id}">
+<!--     <xacro:ar_tag prefix="${prefix}holder_" parent="${prefix}holder_link" tag_id="${tag_id}">
       <origin xyz="0 0 0" rpy="0 0 ${-3.14159/2}"/>
     </xacro:ar_tag>
+ -->
+<!-- Collision bumper -->
+        <joint name="${prefix}holder_right_joint" type="fixed">
+      <origin rpy="0 0 0" xyz="0 -0.10 0.005"/>
+      <parent link="${prefix}holder_base_link"/>
+      <child link="${prefix}holder_right_link"/>
+    </joint>
+    <link name="${prefix}holder_right_link">
+    <inertial>
+      <mass value="0.01" />
+      <origin xyz="0 0 0" rpy="0 0 0" />
+      <solid_cuboid_inertia m="0.01" h="0.01" d="0.26" w="0.01"/>
+    </inertial>
+    <visual>
+      <origin xyz="0 0 0"/>
+      <geometry>
+        <box size="0.26 0.01 0.01" />
+      </geometry>
+    </visual>
+    <collision>
+      <origin xyz="0 0 0"/>
+      <geometry>
+        <box size="0.26 0.01 0.01" />
+      </geometry>
+    </collision>
+    </link>
+    <joint name="${prefix}holder_left_joint" type="fixed">
+      <origin rpy="0 0 0" xyz="0 +0.10 0.005"/>
+      <parent link="${prefix}holder_base_link"/>
+      <child link="${prefix}holder_left_link"/>
+    </joint>
+    <link name="${prefix}holder_left_link">
+    <inertial>
+      <mass value="0.01" />
+      <origin xyz="0 0 0" rpy="0 0 0" />
+      <solid_cuboid_inertia m="0.01" h="0.01" d="0.26" w="0.01"/>
+    </inertial>
+    <visual>
+      <origin xyz="0 0 0"/>
+      <geometry>
+        <box size="0.26 0.01 0.01" />
+      </geometry>
+    </visual>
+    <collision>
+      <origin xyz="0 0 0"/>
+      <geometry>
+        <box size="0.26 0.01 0.01" />
+      </geometry>
+    </collision>
+    </link>
+    <joint name="${prefix}holder_top_joint" type="fixed">
+      <origin rpy="0 0 0" xyz="0.145 0 0.005"/>
+      <parent link="${prefix}holder_base_link"/>
+      <child link="${prefix}holder_top_link"/>
+    </joint>
+    <link name="${prefix}holder_top_link">
+    <inertial>
+      <mass value="0.01" />
+      <origin xyz="0 0 0" rpy="0 0 0" />
+      <solid_cuboid_inertia m="0.01" h="0.01" d="0.01" w="0.16"/>
+    </inertial>
+    <visual>
+      <origin xyz="0 0 0"/>
+      <geometry>
+        <box size="0.01 0.16 0.01" />
+      </geometry>
+    </visual>
+    <collision>
+      <origin xyz="0 0 0"/>
+      <geometry>
+        <box size="0.01 0.16 0.01" />
+      </geometry>
+    </collision>
+    </link>
+        <joint name="${prefix}holder_bottom_joint" type="fixed">
+      <origin rpy="0 0 0" xyz="-0.145 0 0.005"/>
+      <parent link="${prefix}holder_base_link"/>
+      <child link="${prefix}holder_bottom_link"/>
+    </joint>
+    <link name="${prefix}holder_bottom_link">
+    <inertial>
+      <mass value="0.01" />
+      <origin xyz="0 0 0" rpy="0 0 0" />
+      <solid_cuboid_inertia m="0.01" h="0.01" d="0.01" w="0.16"/>
+    </inertial>
+    <visual>
+      <origin xyz="0 0 0"/>
+      <geometry>
+        <box size="0.01 0.16 0.01" />
+      </geometry>
+    </visual>
+    <collision>
+      <origin xyz="0 0 0"/>
+      <geometry>
+        <box size="0.01 0.16 0.01" />
+      </geometry>
+    </collision>
+    </link>
     <gazebo reference="${prefix}holder_link">
       <visual>

Commit message: component_sorting_description: add holder bumper collision + add box grab link

File: component_sorting_description/urdf/box/holder.urdf.xacro (robot description, xacro)
@@ -31,10 +31,10 @@
         </geometry>
       </visual>
-      <!--collision>
-        <origin rpy="0 0 0" xyz="0 0 0"/>
+      <collision>
+        <origin rpy="0 0 ${-3.14159/2}" xyz="0 0 -0.005"/>
         <geometry>
-          <mesh filename="package://component_sorting_description/meshes/box/box_holder.stl"/>
+          <mesh filename="package://component_sorting_description/meshes/box/holder_bumper.stl"/>
         </geometry>
-      </collision-->
+      </collision>
     </link>
     <joint name="${prefix}holder_oriented_joint" type="fixed">
@@ -52,5 +52,5 @@
     <link name="${prefix}holder_approach"/>
     <joint name="${prefix}grab_joint" type="fixed">
-      <origin rpy="0 0 0" xyz="0 0 -0.5"/>
+      <origin rpy="0 0 0" xyz="0 0 -0.236"/>
       <parent link="${prefix}holder_oriented_link"/>
       <child link="${prefix}grab_link"/>
@@ -62,6 +62,5 @@
     </xacro:ar_tag>
  -->
-<!-- Collision bumper -->
-        <joint name="${prefix}holder_right_joint" type="fixed">
+  <!--   <joint name="${prefix}holder_right_joint" type="fixed">
       <origin rpy="0 0 0" xyz="0 -0.10 0.005"/>
       <parent link="${prefix}holder_base_link"/>
@@ -159,4 +158,5 @@
     </collision>
     </link>
+ -->
     <gazebo reference="${prefix}holder_link">
       <visual>
