Commit message: component_sorting_description: -changed ar tags definition
component_sorting_simple_sim:
-Launch file to spawn boxes in kairos
-Launch file to spawn boxes in table

File: component_sorting_description/ar_tags/ar_tag.urdf.xacro (robot description, xacro)
@@ -13,10 +13,10 @@
         <inertia ixx="0.00000001" ixy="0.0"  ixz="0.0"  iyy="0.00000001"  iyz="0.0"  izz="0.00000001"/>
       </inertial>
-      <collision >
+<!--       <collision >
         <origin rpy="0  0  0" xyz="0  0  0"/>
         <geometry>
           <box size="0.001 0.14 0.14"/>
         </geometry>
-      </collision>
+      </collision> -->
       <visual >
         <origin rpy="0  0  0" xyz="0  0  0"/>

File: component_sorting_description/ar_tags/ar_tag_border.urdf.xacro (robot description, xacro)
@@ -13,10 +13,10 @@
         <inertia ixx="0.00000001" ixy="0.0"  ixz="0.0"  iyy="0.00000001"  iyz="0.0"  izz="0.00000001"/>
       </inertial>
-      <collision >
+<!--       <collision >
         <origin rpy="0  0  0" xyz="0  0  0"/>
         <geometry>
           <box size="0.001 0.14 0.14"/>
         </geometry>
-      </collision>
+      </collision> -->
       <visual >
         <origin rpy="0  0  0" xyz="0  0  0"/>

File: component_sorting_description/ar_tags/marker1_border_12cm.urdf.xacro (robot description, xacro)
@@ -1,5 +1,5 @@
 <?xml version="1.0" ?>
 <robot name="marker1_border_12cm" xmlns:xacro="http://wiki.ros.org/xacro">
-  <xacro:macro name="ar_tag" params="prefix parent *origin">
+  <xacro:macro name="ar_tag" params="prefix parent id_tag *origin">
     <joint name="${prefix}ar_tag_base_joint" type="fixed">
       <xacro:insert_block name="origin" />
@@ -9,7 +9,7 @@
     <link name="${prefix}ar_tag_base_link">
       <inertial>
-        <mass value="0"/>
+        <mass value="0.01"/>
         <origin rpy="0  0  0" xyz="0  0  0"/>
-        <inertia ixx="0" ixy="0" ixz="0" iyy="0" iyz="0" izz="0"/>
+        <inertia ixx="0.00000001" ixy="0.0"  ixz="0.0"  iyy="0.00000001"  iyz="0.0"  izz="0.00000001"/>
       </inertial>
       <collision >
@@ -27,5 +27,5 @@
     </link>
     <gazebo reference="${prefix}ar_tag_base_link">
-      <material>ARtrack/marker1_border_12cm</material>
+      <material>ARtrack/${id_tag}</material>
     </gazebo>
   </xacro:macro>

File: component_sorting_description/ar_tags/marker2_border_12cm.urdf.xacro (robot description, xacro)
@@ -9,7 +9,7 @@
     <link name="${prefix}ar_tag_base_link">
       <inertial>
-        <mass value="0"/>
+        <mass value="0.01"/>
         <origin rpy="0  0  0" xyz="0  0  0"/>
-        <inertia ixx="0" ixy="0" ixz="0" iyy="0" iyz="0" izz="0"/>
+        <inertia ixx="0.00000001" ixy="0.0"  ixz="0.0"  iyy="0.00000001"  iyz="0.0"  izz="0.00000001"/>
       </inertial>
       <collision >

File: component_sorting_description/robots/component_sorting.urdf.xacro (robot description, xacro)
@@ -36,4 +36,25 @@
     <!-- ROBOT -->
     <xacro:rbkairos_ur5_oem_vgc10 prefix="$(arg prefix)" publish_bf="true" hq="true" load_kinematics_file="$(arg load_kinematics_file)"/>
+<!--     <joint name="${prefix}base_boxes" type="fixed">
+      <origin rpy="0 0 0" xyz="0 0 0"/>
+      <parent link="${prefix}base_chapa"/>
+      <child link="${prefix}base_boxes_link"/>
+    </joint>
+    <link name="${prefix}base_boxes_link">
+      <collision>
+        <origin xyz="0 0 0.0015"/>
+        <geometry>
+          <box size="0.71 0.57 0.003" />
+        </geometry>
+      </collision>
+    </link>
+    <gazebo reference="${prefix}base_boxes_link">
+      <material>Gazebo/White</material>
+      <mu1>1000000.0</mu1>
+      <mu2>1000000.0</mu2>
+      <kp>10000000.0</kp>
+      <kd>1.0</kd>
+      <minDepth>0.001</minDepth>
+    </gazebo> -->
     <!-- HOLDERS -->
     <xacro:holder_robot prefix="${prefix}center_" parent="${prefix}base_link" tag_id="marker3_border_12cm">

File: component_sorting_description/urdf/box/box.urdf.xacro (robot description, xacro)
@@ -2,5 +2,5 @@
 <robot name="box" xmlns:xacro="http://wiki.ros.org/xacro">
   <xacro:include filename="$(find component_sorting_description)/urdf/inertia.urdf.xacro" />
-  <xacro:include filename="$(find component_sorting_description)/ar_tags/ar_tag.urdf.xacro" />
+  <xacro:include filename="$(find component_sorting_description)/ar_tags/ar_tag_border.urdf.xacro" />
   <xacro:arg name="prefix" default="box_"/>
   <xacro:property name="prefix" value="$(arg prefix)" />
@@ -16,7 +16,7 @@
   <link name="${prefix}body_box_link">
     <inertial>
-      <mass value="5" />
+      <mass value="4" />
       <origin xyz="0 0 0.05" />
-      <solid_cuboid_inertia m="5" h="0.2" d="0.1" w="0.3"/>
+      <solid_cuboid_inertia m="4" h="0.2" d="0.1" w="0.3"/>
     </inertial>
     <visual>
@@ -31,12 +31,4 @@
         <mesh filename="package://component_sorting_description/meshes/box/box_base.stl"/>
       </geometry>
-       <surface>
-        <friction>
-          <ode>
-            <mu>0.01</mu>
-            <mu2>0.01</mu2>
-          </ode>
-        </friction>
-      </surface>
     </collision>
   </link>
@@ -89,4 +81,9 @@
       </material>
     </visual>
+    <mu1>50.0</mu1>
+    <mu2>50.0</mu2>
+    <kp>10000000.0</kp>
+    <kd>1.0</kd>
+<!--     <minDepth>0.002</minDepth> -->
  </gazebo>
   <gazebo reference="${prefix}handle_link">

File: component_sorting_description/urdf/box/holder_robot.urdf.xacro (robot description, xacro)
@@ -30,13 +30,13 @@
         </geometry>
       </visual>
-<!--       <collision>
+      <collision>
         <origin rpy="0 0 0" xyz="0 0 0"/>
         <geometry>
           <mesh filename="package://component_sorting_description/meshes/box/box_holder.stl"/>
         </geometry>
-      </collision>  -->
+      </collision>
     </link>
     <joint name="${prefix}approach_joint" type="fixed">
-      <origin rpy="3.1416 0 0" xyz="0 0 0.691"/>
+      <origin rpy="3.1416 0 0" xyz="-0.075 0 0.741"/>
       <parent link="${prefix}holder_link"/>
       <child link="${prefix}approach"/>
@@ -44,5 +44,5 @@
     <link name="${prefix}approach"/>
     <joint name="${prefix}grab_joint" type="fixed">
-      <origin rpy="3.1416 0 0" xyz="0 0 0.371"/>
+      <origin rpy="3.1416 0 0" xyz="0.0 0 0.371"/>
       <parent link="${prefix}holder_link"/>
       <child link="${prefix}grab"/>

File: component_sorting_description/urdf/box/holder_table.urdf.xacro (robot description, xacro)
@@ -22,5 +22,6 @@
         <mass value="0.1" />
         <origin xyz="0 0.011 0" />
-        <solid_cuboid_inertia m="0.1" h="0.022" d="0.225" w="0.31"/>
+        <xacro:solid_cuboid_inertia m="0.1" h="0.022" d="0.225" w="0.31">
+        </xacro:solid_cuboid_inertia>
       </inertial>
       <visual>
@@ -38,5 +39,5 @@
     </link>
     <joint name="${prefix}approach_joint" type="fixed">
-      <origin rpy="3.1416 0 0" xyz="0 0 0.47"/>
+      <origin rpy="3.1416 0 0" xyz="-0.137 0 0.50"/>
       <parent link="${prefix}holder_link"/>
       <child link="${prefix}approach"/>

File: component_sorting_description/urdf/table.urdf.xacro (robot description, xacro)
@@ -34,4 +34,5 @@
     </plugin>
   </gazebo>
+  <static>true</static>
   <link name="${prefix}qr">
   </link>
@@ -43,7 +44,7 @@
   <link name="${prefix}base_link">
     <inertial>
-      <mass value="40" />
-      <origin xyz="0 0 ${table_height/2}" />
-      <solid_cuboid_inertia m="40" h="${table_height}" d="${table_length}" w="${table_width}"/>
+      <mass value="90" />
+      <origin xyz="0 0 ${table_height/2}" rpy="0 0 0" />
+      <solid_cuboid_inertia m="70" h="${table_height}" d="${table_length}" w="${table_width}"/>
     </inertial>
     <visual>
@@ -58,5 +59,5 @@
         <box size="${table_length} ${table_width} ${table_height}" />
       </geometry>
-      </collision>
+    </collision>
   </link>
         <!-- TABLE TAG -->
@@ -83,6 +84,10 @@
       <origin xyz="${right_holder_offset_x} ${right_holder_offset_y} ${right_holder_offset_z}" rpy="0 0 0"/>
   </xacro:holder_table>
-  <gazebo reference="${prefix}">
-    <material>Gazebo/Grey</material>
+  <gazebo reference="${prefix}base_link">
+    <material>Gazebo/White</material>
+    <mu1>50.0</mu1>
+    <mu2>50.0</mu2>
+    <kp>10000000.0</kp>
+    <kd>1.0</kd>
   </gazebo>
 </robot>

Commit message: component_sorting: Code parametrization
component_sorting_description: Code parametrization

component_sorting_simple_sim: Code parametrization

File: component_sorting_description/ar_tags/ar_tag.urdf.xacro (robot description, xacro)
@@ -9,5 +9,5 @@
     <link name="${prefix}ar_tag_base_link">
       <inertial>
-        <mass value="0.01"/>
+        <mass value="0.00001"/>
         <origin rpy="0  0  0" xyz="0  0  0"/>
         <inertia ixx="0.00000001" ixy="0.0"  ixz="0.0"  iyy="0.00000001"  iyz="0.0"  izz="0.00000001"/>

File: component_sorting_description/ar_tags/ar_tag_12cm_border.urdf.xacro (robot description, xacro)
@@ -9,5 +9,5 @@
     <link name="${prefix}ar_tag_base_link">
       <inertial>
-        <mass value="0.01"/>
+        <mass value="0.00001"/>
         <origin rpy="0  0  0" xyz="0  0  0"/>
         <inertia ixx="0.00000001" ixy="0.0"  ixz="0.0"  iyy="0.00000001"  iyz="0.0"  izz="0.00000001"/>
@@ -33,5 +33,5 @@
     <link name="${prefix}ar_tag_link">
       <inertial>
-        <mass value="0.01"/>
+        <mass value="0.00001"/>
         <origin rpy="0  0  0" xyz="0  0  0"/>
         <inertia ixx="0.00000001" ixy="0.0"  ixz="0.0"  iyy="0.00000001"  iyz="0.0"  izz="0.00000001"/>

File: component_sorting_description/ar_tags/ar_tag_6cm_border.urdf.xacro (robot description, xacro)
@@ -9,5 +9,5 @@
     <link name="${prefix}ar_tag_base_link">
       <inertial>
-        <mass value="0.01"/>
+        <mass value="0.00001"/>
         <origin rpy="0  0  0" xyz="0  0  0"/>
         <inertia ixx="0.00000001" ixy="0.0"  ixz="0.0"  iyy="0.00000001"  iyz="0.0"  izz="0.00000001"/>
@@ -33,5 +33,5 @@
     <link name="${prefix}ar_tag_link">
       <inertial>
-        <mass value="0.01"/>
+        <mass value="0.00001"/>
         <origin rpy="0  0  0" xyz="0  0  0"/>
         <inertia ixx="0.00000001" ixy="0.0"  ixz="0.0"  iyy="0.00000001"  iyz="0.0"  izz="0.00000001"/>

File: component_sorting_description/ar_tags/ar_tag_border.urdf.xacro (robot description, xacro)
@@ -9,5 +9,5 @@
     <link name="${prefix}ar_tag_base_link">
       <inertial>
-        <mass value="0.01"/>
+        <mass value="0.00001"/>
         <origin rpy="0  0  0" xyz="0  0  0"/>
         <inertia ixx="0.00000001" ixy="0.0"  ixz="0.0"  iyy="0.00000001"  iyz="0.0"  izz="0.00000001"/>
@@ -33,5 +33,5 @@
     <link name="${prefix}ar_tag_link">
       <inertial>
-        <mass value="0.01"/>
+        <mass value="0.00001"/>
         <origin rpy="0  0  0" xyz="0  0  0"/>
         <inertia ixx="0.00000001" ixy="0.0"  ixz="0.0"  iyy="0.00000001"  iyz="0.0"  izz="0.00000001"/>

File: component_sorting_description/urdf/box/box.urdf.xacro (robot description, xacro)
@@ -7,4 +7,5 @@
   <xacro:arg name="tag_id" default="1"/>
   <xacro:property name="tag_id" value="$(arg tag_id)" />
+ <allow_auto_disable>false</allow_auto_disable>
   <link name="${prefix}base_link">
   </link>
@@ -31,15 +32,24 @@
         <mesh filename="package://component_sorting_description/meshes/box/box_base.stl"/>
       </geometry>
-<!--         <surface>
-            <friction>
-                <ode>
-                    <mu>200</mu>
-                    <mu2>200</mu2>
-                    <fdir1>0 0 1</fdir1>
-                    <slip1>0</slip1>
-                    <slip2>0</slip2>
-                </ode>
-            </friction>
-        </surface> -->
+<surface>
+      <friction>
+        <ode>
+          <mu>1</mu>
+          <mu2>1</mu2>
+          <slip1>0</slip1>
+          <slip2>0</slip2>
+        </ode>
+      </friction>
+      <contact>
+        <ode>
+          <soft_cfm>0</soft_cfm>
+          <soft_erp>0.2</soft_erp>
+          <kp>1e+13</kp>
+          <kd>1</kd>
+          <max_vel>0.01</max_vel>
+          <min_depth>0</min_depth>
+        </ode>
+      </contact>
+    </surface>
     </collision>
   </link>
@@ -92,9 +102,10 @@
       </material>
     </visual>
-    <mu1>200.0</mu1>
-    <mu2>200.0</mu2>
+    <mu1>1.0</mu1>
+    <mu2>1.0</mu2>
     <kp>10000000.0</kp>
     <kd>1.0</kd>
-     <minDepth>0.001</minDepth>
+   <minDepth>0.001</minDepth>
+   <maxVel>0</maxVel>
     <maxContacts>10</maxContacts>
  </gazebo>

File: component_sorting_description/urdf/table.urdf.xacro (robot description, xacro)
@@ -7,16 +7,18 @@
   <xacro:arg name="prefix" default="table_"/>
   <xacro:property name="prefix" value="$(arg prefix)" />
+  <xacro:property name="yaml_file" value="$(find component_sorting)/config/component_sorting.yaml" />
+  <xacro:property name="component_sorting" value="${load_yaml(yaml_file)}"/>
   <xacro:arg name="table_length" default="0.63"/>
-  <xacro:property name="table_length" value="$(arg table_length)" />
+  <xacro:property name="table_length" value="${component_sorting['table_length']}" />
   <xacro:arg name="table_width" default="0.63"/>
-  <xacro:property name="table_width" value="$(arg table_width)" />
+  <xacro:property name="table_width" value="${component_sorting['table_width']}" />
   <xacro:arg name="table_height" default="0.75"/>
-  <xacro:property name="table_height" value="$(arg table_height)" />
+  <xacro:property name="table_height" value="${component_sorting['table_height']}" />
   <xacro:arg name="holder_width" default="0.228"/>
-  <xacro:property name="holder_width" value="$(arg holder_width)" />
+  <xacro:property name="holder_width" value="${component_sorting['holder_width']}" />
   <xacro:arg name="holder_length" default="0.30"/>
-  <xacro:property name="holder_length" value="$(arg holder_length)" />
+  <xacro:property name="holder_length" value="${component_sorting['holder_length']}" />
   <xacro:arg name="qr_height" default="0.375"/>
-  <xacro:property name="qr_height" value="$(arg qr_height)" />
+  <xacro:property name="qr_height" value="${component_sorting['qr_height']}" />
   <gazebo>
     <plugin name="${prefix}tf_publisher" filename="librobotnik_gazebo_ground_truth_odom.so">
@@ -38,5 +40,5 @@
   </link>
   <joint name="${prefix}base_joint" type="fixed">
-    <origin rpy="0 0 0" xyz="${table_length/2}  0 ${-qr_height+(table_height/2)}"/>
+    <origin rpy="0 0 0" xyz="${table_length/2}  0 ${-qr_height}"/>
     <parent link="${prefix}qr"/>
     <child link="${prefix}base_link"/>
@@ -44,10 +46,10 @@
   <link name="${prefix}base_link">
     <inertial>
-      <mass value="90" />
-      <origin xyz="0 0 0" rpy="0 0 0" />
+      <mass value="70" />
+      <origin xyz="0 0 ${table_height/2}" rpy="0 0 0" />
       <solid_cuboid_inertia m="70" h="${table_height}" d="${table_length}" w="${table_width}"/>
     </inertial>
     <visual>
-      <origin xyz="0 0 0"/>
+      <origin xyz="0 0 ${table_height/2}"/>
       <geometry>
         <box size="${table_length} ${table_width} ${table_height}" />
@@ -55,5 +57,5 @@
     </visual>
     <collision>
-      <origin xyz="0 0 0"/>
+      <origin xyz="0 0 ${table_height/2}"/>
       <geometry>
         <box size="${table_length} ${table_width} ${table_height}" />
@@ -67,11 +69,11 @@
   <xacro:property name="center_holder_offset_x" value="${(holder_length-table_length)/2}"/>
   <xacro:property name="center_holder_offset_y" value="0.0"/>
-  <xacro:property name="center_holder_offset_z" value="${table_height/2}"/>
+  <xacro:property name="center_holder_offset_z" value="${table_height}"/>
   <xacro:property name="left_holder_offset_x" value="${(holder_length-table_length)/2}"/> <!-- -0.195 -->
   <xacro:property name="left_holder_offset_y" value="${holder_width}"/> <!-- 0.225 -->
-  <xacro:property name="left_holder_offset_z" value="${table_height/2}"/>
+  <xacro:property name="left_holder_offset_z" value="${table_height}"/>
   <xacro:property name="right_holder_offset_x" value="${(holder_length-table_length)/2}"/>
   <xacro:property name="right_holder_offset_y" value="${-holder_width}"/>
-  <xacro:property name="right_holder_offset_z" value="${table_height/2}"/>
+  <xacro:property name="right_holder_offset_z" value="${table_height}"/>
     <!-- HOLDERS -->
   <xacro:holder_table prefix="${prefix}center_" parent="${prefix}base_link" tag_id="marker2_12cm" >
