Commit message: component_sorting: -Changed grab position to qr box link -Changed place position to corresponding qr holder link.
component_sorting_bringup:
-Changed qr id names.

component_sorting_description:
-Added qr markers.

Added gazebo_ros_link_attacher

File: component_sorting_description/ar_tags/ar_tag_12cm_border.urdf.xacro (robot description, xacro)
@@ -27,5 +27,5 @@
     </link>
     <joint name="${prefix}ar_tag_joint" type="fixed">
-      <origin rpy="0 0 0" xyz="0 0 0.001"/>
+      <origin rpy="0 0 0" xyz="0 0 0.0005"/>
       <parent link="${prefix}ar_tag_base_link"/>
       <child link="${prefix}ar_tag_link"/>

File: component_sorting_description/ar_tags/ar_tag_6cm_border.urdf.xacro (robot description, xacro)
@@ -22,10 +22,10 @@
         <origin rpy="0  0  0" xyz="0  0  0"/>
         <geometry>
-          <box size="0.14 0.14 0.001"/>
+          <box size="0.08 0.08 0.001"/>
         </geometry>
       </visual>
     </link>
     <joint name="${prefix}ar_tag_joint" type="fixed">
-      <origin rpy="0 0 0" xyz="0 0 0.001"/>
+      <origin rpy="0 0 0" xyz="0 0 0.0005"/>
       <parent link="${prefix}ar_tag_base_link"/>
       <child link="${prefix}ar_tag_link"/>
@@ -46,5 +46,5 @@
         <origin rpy="0  0  0" xyz="0  0  0"/>
         <geometry>
-          <box size="0.12 0.12 0.001"/>
+          <box size="0.06 0.06 0.001"/>
         </geometry>
       </visual>

File: component_sorting_description/robots/component_sorting.urdf.xacro (robot description, xacro)
@@ -58,23 +58,13 @@
     </gazebo> -->
     <!-- HOLDERS -->
-    <xacro:holder_robot prefix="${prefix}center_" parent="${prefix}base_link" tag_id="marker3_border_12cm">
+     <xacro:holder_robot prefix="${prefix}center_" parent="${prefix}base_link" tag_id="marker5_12cm">
         <origin xyz="${center_holder_offset_x} ${center_holder_offset_y} ${center_holder_offset_z}" rpy="0 0 3.14159"/>
     </xacro:holder_robot>
-    <xacro:holder_robot prefix="${prefix}left_" parent="${prefix}base_link" tag_id="marker4_border_12cm">
+    <xacro:holder_robot prefix="${prefix}left_" parent="${prefix}base_link" tag_id="marker6_12cm">
         <origin xyz="${left_holder_offset_x} ${left_holder_offset_y} ${left_holder_offset_z}" rpy="0 0 3.14159"/>
     </xacro:holder_robot>
-    <xacro:holder_robot prefix="${prefix}right_" parent="${prefix}base_link" tag_id="marker2_border_12cm" >
+    <xacro:holder_robot prefix="${prefix}right_" parent="${prefix}base_link" tag_id="marker4_12cm" >
         <origin xyz="${right_holder_offset_x} ${right_holder_offset_y} ${right_holder_offset_z}" rpy="0 0 3.14159"/>
     </xacro:holder_robot>
-    <!-- HOLDERS TABLE-->
-<!--     <xacro:test prefix="${prefix}center_table_" parent="${prefix}base_footprint">
-        <origin xyz="${center_table_holder_offset_x} ${center_table_holder_offset_y} ${center_table_holder_offset_z}" rpy="0 0 3.14"/>
-    </xacro:test>
-    <xacro:test prefix="${prefix}left_table_" parent="${prefix}base_footprint">
-        <origin xyz="${left_table_holder_offset_x} ${left_table_holder_offset_y} ${left_table_holder_offset_z}" rpy="0 0 3.14"/>
-    </xacro:test>
-    <xacro:test prefix="${prefix}right_table_" parent="${prefix}base_footprint">
-        <origin xyz="${right_table_holder_offset_x} ${right_table_holder_offset_y} ${right_table_holder_offset_z}" rpy="0 0 3.14"/>
-    </xacro:test> -->
     <!-- BOX -->
 <!--   <joint name="${prefix}joint" type="fixed">

File: component_sorting_description/urdf/box/box.urdf.xacro (robot description, xacro)
@@ -2,5 +2,5 @@
 <robot name="box" xmlns:xacro="http://wiki.ros.org/xacro">
   <xacro:include filename="$(find component_sorting_description)/urdf/inertia.urdf.xacro" />
-  <xacro:include filename="$(find component_sorting_description)/ar_tags/ar_tag_border.urdf.xacro" />
+  <xacro:include filename="$(find component_sorting_description)/ar_tags/ar_tag_6cm_border.urdf.xacro" />
   <xacro:arg name="prefix" default="box_"/>
   <xacro:property name="prefix" value="$(arg prefix)" />
@@ -31,9 +31,20 @@
         <mesh filename="package://component_sorting_description/meshes/box/box_base.stl"/>
       </geometry>
+<!--         <surface>
+            <friction>
+                <ode>
+                    <mu>200</mu>
+                    <mu2>200</mu2>
+                    <fdir1>0 0 1</fdir1>
+                    <slip1>0</slip1>
+                    <slip2>0</slip2>
+                </ode>
+            </friction>
+        </surface> -->
     </collision>
   </link>
   <joint name="${prefix}handle_joint" type="prismatic">
     <axis xyz="0 0 1"/>
-    <limit effort="1000.0" lower="-0.03" upper="0.03" velocity="0.5"/>
+    <limit effort="1000.0" lower="-0.025" upper="0.025" velocity="0.5"/>
     <origin rpy="0 0 0" xyz="0 0 0.1"/>
     <parent link="${prefix}body_box_link"/>
@@ -66,6 +77,6 @@
   <link name="${prefix}grasping_link"/>
   <!-- AR TAG -->
-  <xacro:ar_tag prefix="${prefix}" parent="${prefix}grasping_link" tag_id="${tag_id}">
-    <origin xyz="-0.001 0  0" rpy="0 ${3.14159/2} 0"/>
+  <xacro:ar_tag prefix="${prefix}" parent="${prefix}handle_link" tag_id="${tag_id}">
+    <origin xyz="0 0 0.1575" rpy="0 0 0"/>
   </xacro:ar_tag>
 <!--  <xacro:artag name="artag_01" parent="${prefix}grasping_link">
@@ -81,9 +92,10 @@
       </material>
     </visual>
-    <mu1>50.0</mu1>
-    <mu2>50.0</mu2>
+    <mu1>200.0</mu1>
+    <mu2>200.0</mu2>
     <kp>10000000.0</kp>
     <kd>1.0</kd>
-<!--     <minDepth>0.002</minDepth> -->
+     <minDepth>0.001</minDepth>
+    <maxContacts>10</maxContacts>
  </gazebo>
   <gazebo reference="${prefix}handle_link">

File: component_sorting_description/urdf/box/holder_robot.urdf.xacro (robot description, xacro)
@@ -2,5 +2,5 @@
 <robot name="holder" xmlns:xacro="http://wiki.ros.org/xacro">
   <xacro:include filename="$(find component_sorting_description)/urdf/inertia.urdf.xacro" />
-  <xacro:include filename="$(find component_sorting_description)/ar_tags/ar_tag_border.urdf.xacro" />
+  <xacro:include filename="$(find component_sorting_description)/ar_tags/ar_tag_12cm_border.urdf.xacro" />
   <!--xacro:arg name="prefix" default="box_"/>
   <xacro:property name="prefix" value="$(arg prefix)" /-->
@@ -51,5 +51,5 @@
     <!-- TABLE TAG -->
     <xacro:ar_tag prefix="${prefix}" parent="${prefix}holder_link" tag_id="${tag_id}">
-      <origin xyz="0.001 0 0" rpy="0 ${3.14159/2} 0"/>
+      <origin xyz="0 0 0" rpy="0 0 0"/>
     </xacro:ar_tag>
     <gazebo reference="${prefix}holder_link">

File: component_sorting_description/urdf/box/holder_table.urdf.xacro (robot description, xacro)
@@ -2,5 +2,5 @@
 <robot name="holder" xmlns:xacro="http://wiki.ros.org/xacro">
   <xacro:include filename="$(find component_sorting_description)/urdf/inertia.urdf.xacro" />
-  <xacro:include filename="$(find component_sorting_description)/ar_tags/ar_tag_border.urdf.xacro" />
+  <xacro:include filename="$(find component_sorting_description)/ar_tags/ar_tag_12cm_border.urdf.xacro" />
   <!--xacro:arg name="prefix" default="box_"/>
   <xacro:property name="prefix" value="$(arg prefix)" /-->
@@ -51,6 +51,6 @@
     <link name="${prefix}grab"/>
     <!-- TABLE TAG -->
-    <xacro:ar_tag prefix="${prefix}" parent="${prefix}holder_link" tag_id="${tag_id}">
-      <origin xyz="0.001 0 0" rpy="0 ${3.14159/2} 0"/>
+    <xacro:ar_tag prefix="${prefix}holder_" parent="${prefix}holder_link" tag_id="${tag_id}">
+      <origin xyz="0 0 0" rpy="0 0 0"/>
     </xacro:ar_tag>
     <gazebo reference="${prefix}holder_link">

File: component_sorting_description/urdf/table.urdf.xacro (robot description, xacro)
@@ -4,5 +4,5 @@
   <xacro:include filename="$(find component_sorting_description)/urdf/box/holder_table.urdf.xacro" />
 <!--   <xacro:include filename="$(find vigir_ar_alvar_description)/urdf/artag.urdf.xacro" /> -->
-  <xacro:include filename="$(find component_sorting_description)/ar_tags/ar_tag_border.urdf.xacro" />
+  <xacro:include filename="$(find component_sorting_description)/ar_tags/ar_tag_12cm_border.urdf.xacro" />
   <xacro:arg name="prefix" default="table_"/>
   <xacro:property name="prefix" value="$(arg prefix)" />
@@ -38,5 +38,5 @@
   </link>
   <joint name="${prefix}base_joint" type="fixed">
-    <origin rpy="0 0 0" xyz="${table_length/2}  0 ${-qr_height}"/>
+    <origin rpy="0 0 0" xyz="${table_length/2}  0 ${-qr_height+(table_height/2)}"/>
     <parent link="${prefix}qr"/>
     <child link="${prefix}base_link"/>
@@ -45,9 +45,9 @@
     <inertial>
       <mass value="90" />
-      <origin xyz="0 0 ${table_height/2}" rpy="0 0 0" />
+      <origin xyz="0 0 0" rpy="0 0 0" />
       <solid_cuboid_inertia m="70" h="${table_height}" d="${table_length}" w="${table_width}"/>
     </inertial>
     <visual>
-      <origin xyz="0 0 ${table_height/2}"/>
+      <origin xyz="0 0 0"/>
       <geometry>
         <box size="${table_length} ${table_width} ${table_height}" />
@@ -55,5 +55,5 @@
     </visual>
     <collision>
-      <origin xyz="0 0 ${table_height/2}"/>
+      <origin xyz="0 0 0"/>
       <geometry>
         <box size="${table_length} ${table_width} ${table_height}" />
@@ -62,24 +62,24 @@
   </link>
         <!-- TABLE TAG -->
-  <xacro:ar_tag prefix="${prefix}" parent="${prefix}qr" tag_id="marker1_border_12cm">
-      <origin xyz="-0.001 0 0" rpy="3.14159 3.14159 0"/>
+  <xacro:ar_tag prefix="${prefix}" parent="${prefix}qr" tag_id="marker10_12cm">
+      <origin xyz="0 0 0" rpy="0 ${-3.14159/2} 0"/>
   </xacro:ar_tag>
   <xacro:property name="center_holder_offset_x" value="${(holder_length-table_length)/2}"/>
   <xacro:property name="center_holder_offset_y" value="0.0"/>
-  <xacro:property name="center_holder_offset_z" value="${table_height}"/>
+  <xacro:property name="center_holder_offset_z" value="${table_height/2}"/>
   <xacro:property name="left_holder_offset_x" value="${(holder_length-table_length)/2}"/> <!-- -0.195 -->
   <xacro:property name="left_holder_offset_y" value="${holder_width}"/> <!-- 0.225 -->
-  <xacro:property name="left_holder_offset_z" value="${table_height}"/>
+  <xacro:property name="left_holder_offset_z" value="${table_height/2}"/>
   <xacro:property name="right_holder_offset_x" value="${(holder_length-table_length)/2}"/>
   <xacro:property name="right_holder_offset_y" value="${-holder_width}"/>
-  <xacro:property name="right_holder_offset_z" value="${table_height}"/>
+  <xacro:property name="right_holder_offset_z" value="${table_height/2}"/>
     <!-- HOLDERS -->
-  <xacro:holder_table prefix="${prefix}center_" parent="${prefix}base_link" tag_id="marker3_border_12cm" >
+  <xacro:holder_table prefix="${prefix}center_" parent="${prefix}base_link" tag_id="marker2_12cm" >
       <origin xyz="${center_holder_offset_x} ${center_holder_offset_y} ${center_holder_offset_z}" rpy="0 0 0"/>
   </xacro:holder_table>
-  <xacro:holder_table prefix="${prefix}left_" parent="${prefix}base_link" tag_id="marker4_border_12cm" >
+  <xacro:holder_table prefix="${prefix}left_" parent="${prefix}base_link" tag_id="marker3_12cm" >
       <origin xyz="${left_holder_offset_x} ${left_holder_offset_y} ${left_holder_offset_z}" rpy="0 0 0"/>
   </xacro:holder_table>
-  <xacro:holder_table prefix="${prefix}right_" parent="${prefix}base_link" tag_id="marker2_border_12cm" >
+  <xacro:holder_table prefix="${prefix}right_" parent="${prefix}base_link" tag_id="marker1_12cm" >
       <origin xyz="${right_holder_offset_x} ${right_holder_offset_y} ${right_holder_offset_z}" rpy="0 0 0"/>
   </xacro:holder_table>

Commit message: component_sorting_description: modify ar_tag urdfs so that they have the same orientation as the qr code frame located by the camera_locator node

File: component_sorting_description/ar_tags/ar_tag_12cm_border.urdf.xacro (robot description, xacro)
@@ -27,5 +27,5 @@
     </link>
     <joint name="${prefix}ar_tag_joint" type="fixed">
-      <origin rpy="0 0 0" xyz="0 0 0.0005"/>
+      <origin rpy="0 0 ${+3.14159/2}" xyz="0 0 0.0005"/>
       <parent link="${prefix}ar_tag_base_link"/>
       <child link="${prefix}ar_tag_link"/>

File: component_sorting_description/ar_tags/ar_tag_6cm_border.urdf.xacro (robot description, xacro)
@@ -27,5 +27,5 @@
     </link>
     <joint name="${prefix}ar_tag_joint" type="fixed">
-      <origin rpy="0 0 0" xyz="0 0 0.0005"/>
+      <origin rpy="0 0 ${+3.14159/2}" xyz="0 0 0.0005"/>
       <parent link="${prefix}ar_tag_base_link"/>
       <child link="${prefix}ar_tag_link"/>
