Commit message: component_sorting_description: -Added a global ar_tag.urdf.xacro
component_sorting_sim:
-Added boxes launcher

component_sorting_description:
-Created box urdf with qr tag to spawn in gazebo

File: component_sorting_description/robots/component_sorting.urdf.xacro (robot description, xacro)
@@ -9,28 +9,105 @@
   	<xacro:arg name="prefix" default="robot_"/>
     <xacro:property name="prefix" value="$(arg prefix)" />
-    <xacro:include filename="$(find rbkairos_description)/robots/versions/rbkairos_ur5_oem_vgc10.urdf.xacro" />
+    <!--xacro:include filename="$(find rbkairos_description)/robots/versions/rbkairos_ur5_oem_vgc10.urdf.xacro" /-->
+    <xacro:include filename="$(find rbkairos_description)/robots/versions/rbkairos_ur5_vgc10.urdf.xacro" />
     <!-- Import holder for the boxes -->
 	<xacro:include filename="$(find rbkairos_description)/urdf/box/holder.urdf.xacro" />
+    <!-- Import  holder for the boxes test -->
+	<xacro:include filename="$(find component_sorting_description)/urdf/box/holder_robot.urdf.xacro" />
     <!-- Holder parameters -->
-    <xacro:property name="center_holder_offset_x" value="-0.195"/>
+    <xacro:property name="center_holder_offset_x" value="-0.2025"/>
     <xacro:property name="center_holder_offset_y" value="0.0"/>
-    <xacro:property name="center_holder_offset_z" value="0.56162"/>
-    <xacro:property name="left_holder_offset_x" value="-0.195"/>
-    <xacro:property name="left_holder_offset_y" value="0.225"/>
-    <xacro:property name="left_holder_offset_z" value="0.56162"/>
-    <xacro:property name="right_holder_offset_x" value="-0.195"/>
-    <xacro:property name="right_holder_offset_y" value="-0.225"/>
-    <xacro:property name="right_holder_offset_z" value="0.56162"/>
+    <xacro:property name="center_holder_offset_z" value="0.38212"/>
+    <xacro:property name="left_holder_offset_x" value="-0.2025"/> <!-- -0.195 -->
+    <xacro:property name="left_holder_offset_y" value="0.228"/> <!-- 0.225 -->
+    <xacro:property name="left_holder_offset_z" value="0.38212"/>
+    <xacro:property name="right_holder_offset_x" value="-0.2025"/>
+    <xacro:property name="right_holder_offset_y" value="-0.228"/>
+    <xacro:property name="right_holder_offset_z" value="0.38212"/>
+    <xacro:property name="center_table_holder_offset_x" value="0.68"/>
+    <xacro:property name="center_table_holder_offset_y" value="0.0"/>
+    <xacro:property name="center_table_holder_offset_z" value="0.9"/>
+    <xacro:property name="left_table_holder_offset_x" value="0.68"/>
+    <xacro:property name="left_table_holder_offset_y" value="0.228"/>
+    <xacro:property name="left_table_holder_offset_z" value="0.9"/>
+    <xacro:property name="right_table_holder_offset_x" value="0.68"/>
+    <xacro:property name="right_table_holder_offset_y" value="-0.228"/>
+    <xacro:property name="right_table_holder_offset_z" value="0.9"/>
     <!-- ROBOT -->
     <xacro:rbkairos_ur5_oem_vgc10 prefix="$(arg prefix)" publish_bf="true" hq="true" load_kinematics_file="$(arg load_kinematics_file)"/>
     <!-- HOLDERS -->
-    <xacro:holder prefix="${prefix}center_" parent="${prefix}base_link">
-        <origin xyz="${center_holder_offset_x} ${center_holder_offset_y} ${center_holder_offset_z}" rpy="0 0 0"/>
-    </xacro:holder>
-    <xacro:holder prefix="${prefix}left_" parent="${prefix}base_link">
-        <origin xyz="${left_holder_offset_x} ${left_holder_offset_y} ${left_holder_offset_z}" rpy="0 0 0"/>
-    </xacro:holder>
-    <xacro:holder prefix="${prefix}right_" parent="${prefix}base_link">
-        <origin xyz="${right_holder_offset_x} ${right_holder_offset_y} ${right_holder_offset_z}" rpy="0 0 0"/>
-    </xacro:holder>
+    <xacro:holder_robot prefix="${prefix}center_" parent="${prefix}base_link" tag_id="marker3_border_12cm">
+        <origin xyz="${center_holder_offset_x} ${center_holder_offset_y} ${center_holder_offset_z}" rpy="0 0 3.14159"/>
+    </xacro:holder_robot>
+    <xacro:holder_robot prefix="${prefix}left_" parent="${prefix}base_link" tag_id="marker4_border_12cm">
+        <origin xyz="${left_holder_offset_x} ${left_holder_offset_y} ${left_holder_offset_z}" rpy="0 0 3.14159"/>
+    </xacro:holder_robot>
+    <xacro:holder_robot prefix="${prefix}right_" parent="${prefix}base_link" tag_id="marker2_border_12cm" >
+        <origin xyz="${right_holder_offset_x} ${right_holder_offset_y} ${right_holder_offset_z}" rpy="0 0 3.14159"/>
+    </xacro:holder_robot>
+    <!-- HOLDERS TABLE-->
+<!--     <xacro:test prefix="${prefix}center_table_" parent="${prefix}base_footprint">
+        <origin xyz="${center_table_holder_offset_x} ${center_table_holder_offset_y} ${center_table_holder_offset_z}" rpy="0 0 3.14"/>
+    </xacro:test>
+    <xacro:test prefix="${prefix}left_table_" parent="${prefix}base_footprint">
+        <origin xyz="${left_table_holder_offset_x} ${left_table_holder_offset_y} ${left_table_holder_offset_z}" rpy="0 0 3.14"/>
+    </xacro:test>
+    <xacro:test prefix="${prefix}right_table_" parent="${prefix}base_footprint">
+        <origin xyz="${right_table_holder_offset_x} ${right_table_holder_offset_y} ${right_table_holder_offset_z}" rpy="0 0 3.14"/>
+    </xacro:test> -->
+    <!-- BOX -->
+<!--   <joint name="${prefix}joint" type="fixed">
+    <origin rpy="0 0 0" xyz="0 0 0.01"/>
+    <parent link="${prefix}right_table_holder_link"/>
+    <child link="${prefix}body_box_link"/>
+  </joint>
+  <link name="${prefix}body_box_link">
+    <inertial>
+      <mass value="5" />
+      <origin xyz="0 0 0.05" />
+      <solid_cuboid_inertia m="5" h="0.2" d="0.1" w="0.3"/>
+    </inertial>
+    <visual>
+      <origin rpy="0 0 0" xyz="0 0 0"/>
+      <geometry>
+        <mesh filename="package://component_sorting_description/meshes/box/box_base.stl"/>
+      </geometry>
+    </visual>
+    <collision>
+      <origin rpy="0 0 0" xyz="0 0 0"/>
+      <geometry>
+        <mesh filename="package://component_sorting_description/meshes/box/box_base.stl"/>
+      </geometry>
+    </collision>
+  </link>
+  <joint name="${prefix}handle_joint" type="fixed">
+    <origin rpy="0 0 0" xyz="0 0 0.1"/>
+    <parent link="${prefix}body_box_link"/>
+    <child link="${prefix}handle_link"/>
+  </joint>
+  <link name="${prefix}handle_link">
+    <inertial>
+      <mass value="0.1" />
+      <origin xyz="0 0 0" />
+      <solid_cuboid_inertia m="0.1" h="0.2" d="0.01" w="0.3"/>
+    </inertial>
+    <visual>
+      <origin rpy="0 0 0" xyz="0 0 0"/>
+      <geometry>
+        <mesh filename="package://component_sorting_description/meshes/box/handle.stl"/>
+      </geometry>
+    </visual>
+    <collision>
+      <origin rpy="0 0 0" xyz="0 0 0"/>
+      <geometry>
+        <mesh filename="package://component_sorting_description/meshes/box/handle.stl"/>
+      </geometry>
+    </collision>
+  </link>
+  <joint name="${prefix}grasping_joint" type="fixed">
+    <origin rpy="3.141592 0 0" xyz="0 0 0.25"/>
+    <parent link="${prefix}body_box_link"/>
+    <child link="${prefix}grasping_link"/>
+  </joint>
+  <link name="${prefix}grasping_link"/> -->
 </robot>

File: component_sorting_description/urdf/box/box.urdf.xacro (robot description, xacro)
@@ -2,6 +2,9 @@
 <robot name="box" xmlns:xacro="http://wiki.ros.org/xacro">
   <xacro:include filename="$(find component_sorting_description)/urdf/inertia.urdf.xacro" />
+  <xacro:include filename="$(find component_sorting_description)/ar_tags/ar_tag.urdf.xacro" />
   <xacro:arg name="prefix" default="box_"/>
   <xacro:property name="prefix" value="$(arg prefix)" />
+  <xacro:arg name="tag_id" default="1"/>
+  <xacro:property name="tag_id" value="$(arg tag_id)" />
   <link name="${prefix}base_link">
   </link>
@@ -28,7 +31,17 @@
         <mesh filename="package://component_sorting_description/meshes/box/box_base.stl"/>
       </geometry>
+       <surface>
+        <friction>
+          <ode>
+            <mu>0.01</mu>
+            <mu2>0.01</mu2>
+          </ode>
+        </friction>
+      </surface>
     </collision>
   </link>
-  <joint name="${prefix}handle_joint" type="fixed">
+  <joint name="${prefix}handle_joint" type="prismatic">
+    <axis xyz="0 0 1"/>
+    <limit effort="1000.0" lower="-0.03" upper="0.03" velocity="0.5"/>
     <origin rpy="0 0 0" xyz="0 0 0.1"/>
     <parent link="${prefix}body_box_link"/>
@@ -55,28 +68,35 @@
   </link>
   <joint name="${prefix}grasping_joint" type="fixed">
-    <origin rpy="3.141592 0 0" xyz="0 0 0.25"/>
-    <parent link="${prefix}body_box_link"/>
+    <origin rpy="3.141592 0 0" xyz="0 0 0.158"/>
+    <parent link="${prefix}handle_link"/>
     <child link="${prefix}grasping_link"/>
   </joint>
   <link name="${prefix}grasping_link"/>
-      <gazebo reference="${prefix}body_box_link">
-      <visual>
-        <material>
-          <ambient>0.0 0.0 0.0 1.0</ambient>
-          <diffuse>0.2 0.2 0.2 1.0</diffuse>
-          <specular>0.584313725 0.647058824 0.650980392 1.0</specular>
-          <emissive>0.0 0.0 0.0 0.0</emissive>
-        </material>
-      </visual>
-    </gazebo>
-      <gazebo reference="${prefix}handle_link">
-      <visual>
-        <material>
-          <ambient>0.0 0.0 0.0 1.0</ambient>
-          <diffuse>0.2 0.2 0.2 1.0</diffuse>
-          <specular>0.584313725 0.647058824 0.650980392 1.0</specular>
-          <emissive>0.0 0.0 0.0 0.0</emissive>
-        </material>
-      </visual>
-    </gazebo>
+  <!-- AR TAG -->
+  <xacro:ar_tag prefix="${prefix}" parent="${prefix}grasping_link" tag_id="${tag_id}">
+    <origin xyz="-0.001 0  0" rpy="0 ${3.14159/2} 0"/>
+  </xacro:ar_tag>
+<!--  <xacro:artag name="artag_01" parent="${prefix}grasping_link">
+    <origin xyz="0 0 0" rpy="0 3.141592 0"/>
+  </xacro:artag>  -->
+  <gazebo reference="${prefix}body_box_link">
+    <visual>
+      <material>
+        <ambient>0.0 0.0 0.0 1.0</ambient>
+        <diffuse>0.2 0.2 0.2 1.0</diffuse>
+        <specular>0.584313725 0.647058824 0.650980392 1.0</specular>
+        <emissive>0.0 0.0 0.0 0.0</emissive>
+      </material>
+    </visual>
+ </gazebo>
+  <gazebo reference="${prefix}handle_link">
+    <visual>
+      <material>
+        <ambient>0.0 0.0 0.0 1.0</ambient>
+        <diffuse>0.2 0.2 0.2 1.0</diffuse>
+        <specular>0.584313725 0.647058824 0.650980392 1.0</specular>
+        <emissive>0.0 0.0 0.0 0.0</emissive>
+      </material>
+    </visual>
+  </gazebo>
 </robot>

File: component_sorting_description/urdf/box/holder_robot.urdf.xacro (robot description, xacro)
@@ -2,7 +2,8 @@
 <robot name="holder" xmlns:xacro="http://wiki.ros.org/xacro">
   <xacro:include filename="$(find component_sorting_description)/urdf/inertia.urdf.xacro" />
+  <xacro:include filename="$(find component_sorting_description)/ar_tags/ar_tag_border.urdf.xacro" />
   <!--xacro:arg name="prefix" default="box_"/>
   <xacro:property name="prefix" value="$(arg prefix)" /-->
-  <xacro:macro name="holder_robot" params="prefix parent *origin">
+  <xacro:macro name="holder_robot" params="prefix parent tag_id *origin">
     <joint name="${prefix}holder_base_joint" type="fixed">
       <xacro:insert_block name="origin" />
@@ -29,13 +30,13 @@
         </geometry>
       </visual>
-      <collision>
+<!--       <collision>
         <origin rpy="0 0 0" xyz="0 0 0"/>
         <geometry>
           <mesh filename="package://component_sorting_description/meshes/box/box_holder.stl"/>
         </geometry>
-      </collision>
+      </collision>  -->
     </link>
     <joint name="${prefix}approach_joint" type="fixed">
-      <origin rpy="3.1416 0 -3.1416" xyz="0 0 0.691"/>
+      <origin rpy="3.1416 0 0" xyz="0 0 0.691"/>
       <parent link="${prefix}holder_link"/>
       <child link="${prefix}approach"/>
@@ -43,9 +44,13 @@
     <link name="${prefix}approach"/>
     <joint name="${prefix}grab_joint" type="fixed">
-      <origin rpy="3.1416 0 -3.1416" xyz="0 0 0.371"/>
+      <origin rpy="3.1416 0 0" xyz="0 0 0.371"/>
       <parent link="${prefix}holder_link"/>
       <child link="${prefix}grab"/>
     </joint>
     <link name="${prefix}grab"/>
+    <!-- TABLE TAG -->
+    <xacro:ar_tag prefix="${prefix}" parent="${prefix}holder_link" tag_id="${tag_id}">
+      <origin xyz="0.001 0 0" rpy="0 ${3.14159/2} 0"/>
+    </xacro:ar_tag>
     <gazebo reference="${prefix}holder_link">
       <visual>

File: component_sorting_description/urdf/box/holder_table.urdf.xacro (robot description, xacro)
@@ -2,8 +2,8 @@
 <robot name="holder" xmlns:xacro="http://wiki.ros.org/xacro">
   <xacro:include filename="$(find component_sorting_description)/urdf/inertia.urdf.xacro" />
+  <xacro:include filename="$(find component_sorting_description)/ar_tags/ar_tag_border.urdf.xacro" />
   <!--xacro:arg name="prefix" default="box_"/>
   <xacro:property name="prefix" value="$(arg prefix)" /-->
   <xacro:macro name="holder_table" params="prefix parent tag_id *origin">
-    <xacro:include filename="$(find component_sorting_description)/ar_tags/marker${tag_id}_border_12cm.urdf.xacro" />
     <joint name="${prefix}holder_base_joint" type="fixed">
       <xacro:insert_block name="origin" />
@@ -50,7 +50,7 @@
     <link name="${prefix}grab"/>
     <!-- TABLE TAG -->
-  <xacro:ar_tag prefix="${prefix}" parent="${prefix}holder_link">
+    <xacro:ar_tag prefix="${prefix}" parent="${prefix}holder_link" tag_id="${tag_id}">
       <origin xyz="0.001 0 0" rpy="0 ${3.14159/2} 0"/>
-  </xacro:ar_tag>
+    </xacro:ar_tag>
     <gazebo reference="${prefix}holder_link">
       <visual>

File: component_sorting_description/urdf/table.urdf.xacro (robot description, xacro)
@@ -4,5 +4,5 @@
   <xacro:include filename="$(find component_sorting_description)/urdf/box/holder_table.urdf.xacro" />
 <!--   <xacro:include filename="$(find vigir_ar_alvar_description)/urdf/artag.urdf.xacro" /> -->
-  <xacro:include filename="$(find component_sorting_description)/ar_tags/marker1_border_12cm.urdf.xacro" />
+  <xacro:include filename="$(find component_sorting_description)/ar_tags/ar_tag_border.urdf.xacro" />
   <xacro:arg name="prefix" default="table_"/>
   <xacro:property name="prefix" value="$(arg prefix)" />
@@ -61,5 +61,5 @@
   </link>
         <!-- TABLE TAG -->
-  <xacro:ar_tag prefix="table" parent="${prefix}qr">
+  <xacro:ar_tag prefix="${prefix}" parent="${prefix}qr" tag_id="marker1_border_12cm">
       <origin xyz="-0.001 0 0" rpy="3.14159 3.14159 0"/>
   </xacro:ar_tag>
@@ -74,11 +74,11 @@
   <xacro:property name="right_holder_offset_z" value="${table_height}"/>
     <!-- HOLDERS -->
-  <xacro:holder_table prefix="${prefix}center_" parent="${prefix}base_link" tag_id="3" >
+  <xacro:holder_table prefix="${prefix}center_" parent="${prefix}base_link" tag_id="marker3_border_12cm" >
       <origin xyz="${center_holder_offset_x} ${center_holder_offset_y} ${center_holder_offset_z}" rpy="0 0 0"/>
   </xacro:holder_table>
-  <xacro:holder_table prefix="${prefix}left_" parent="${prefix}base_link" tag_id="4" >
+  <xacro:holder_table prefix="${prefix}left_" parent="${prefix}base_link" tag_id="marker4_border_12cm" >
       <origin xyz="${left_holder_offset_x} ${left_holder_offset_y} ${left_holder_offset_z}" rpy="0 0 0"/>
   </xacro:holder_table>
-  <xacro:holder_table prefix="${prefix}right_" parent="${prefix}base_link" tag_id="2" >
+  <xacro:holder_table prefix="${prefix}right_" parent="${prefix}base_link" tag_id="marker2_border_12cm" >
       <origin xyz="${right_holder_offset_x} ${right_holder_offset_y} ${right_holder_offset_z}" rpy="0 0 0"/>
   </xacro:holder_table>

Commit message: component_sorting_description: Unified holder_robot and holder_table urdf into on holder urdf

File: component_sorting_description/robots/component_sorting.urdf.xacro (robot description, xacro)
@@ -12,7 +12,8 @@
     <xacro:include filename="$(find rbkairos_description)/robots/versions/rbkairos_ur5_vgc10.urdf.xacro" />
     <!-- Import holder for the boxes -->
-	<xacro:include filename="$(find rbkairos_description)/urdf/box/holder.urdf.xacro" />
+<!-- 	<xacro:include filename="$(find rbkairos_description)/urdf/box/holder.urdf.xacro" /> -->
     <!-- Import  holder for the boxes test -->
-	<xacro:include filename="$(find component_sorting_description)/urdf/box/holder_robot.urdf.xacro" />
+	<xacro:include filename="$(find component_sorting_description)/urdf/box/holder.urdf.xacro" />
+  <xacro:include filename="$(find component_sorting_description)/urdf/inertia.urdf.xacro" />
     <!-- Holder parameters -->
     <xacro:property name="center_holder_offset_x" value="-0.2025"/>
@@ -58,13 +59,13 @@
     </gazebo> -->
     <!-- HOLDERS -->
-     <xacro:holder_robot prefix="${prefix}center_" parent="${prefix}base_link" tag_id="marker5_12cm">
+     <xacro:holder prefix="${prefix}center_" parent="${prefix}base_link" tag_id="marker5_12cm">
         <origin xyz="${center_holder_offset_x} ${center_holder_offset_y} ${center_holder_offset_z}" rpy="0 0 3.14159"/>
-    </xacro:holder_robot>
-    <xacro:holder_robot prefix="${prefix}left_" parent="${prefix}base_link" tag_id="marker6_12cm">
+    </xacro:holder>
+    <xacro:holder prefix="${prefix}left_" parent="${prefix}base_link" tag_id="marker6_12cm">
         <origin xyz="${left_holder_offset_x} ${left_holder_offset_y} ${left_holder_offset_z}" rpy="0 0 3.14159"/>
-    </xacro:holder_robot>
-    <xacro:holder_robot prefix="${prefix}right_" parent="${prefix}base_link" tag_id="marker4_12cm" >
+    </xacro:holder>
+    <xacro:holder prefix="${prefix}right_" parent="${prefix}base_link" tag_id="marker4_12cm" >
         <origin xyz="${right_holder_offset_x} ${right_holder_offset_y} ${right_holder_offset_z}" rpy="0 0 3.14159"/>
-    </xacro:holder_robot>
+    </xacro:holder>
     <!-- BOX -->
 <!--   <joint name="${prefix}joint" type="fixed">

File: component_sorting_description/urdf/box/holder.urdf.xacro (robot description, xacro)
@@ -2,7 +2,8 @@
 <robot name="holder" xmlns:xacro="http://wiki.ros.org/xacro">
   <xacro:include filename="$(find component_sorting_description)/urdf/inertia.urdf.xacro" />
+  <xacro:include filename="$(find component_sorting_description)/ar_tags/ar_tag_12cm_border.urdf.xacro" />
   <!--xacro:arg name="prefix" default="box_"/>
   <xacro:property name="prefix" value="$(arg prefix)" /-->
-  <xacro:macro name="holder" params="prefix parent *origin">
+  <xacro:macro name="holder" params="prefix parent tag_id *origin">
     <joint name="${prefix}holder_base_joint" type="fixed">
       <xacro:insert_block name="origin" />
@@ -21,5 +22,6 @@
         <mass value="0.1" />
         <origin xyz="0 0.011 0" />
-        <solid_cuboid_inertia m="0.1" h="0.022" d="0.225" w="0.31"/>
+        <xacro:solid_cuboid_inertia m="0.1" h="0.022" d="0.225" w="0.31">
+        </xacro:solid_cuboid_inertia>
       </inertial>
       <visual>
@@ -37,9 +39,19 @@
     </link>
     <joint name="${prefix}holder_approach_joint" type="fixed">
-      <origin rpy="3.1415 0 0" xyz="0 0 0.5"/>
+      <origin rpy="3.1416 0 0" xyz="-0.137 0 0.50"/>
       <parent link="${prefix}holder_link"/>
-      <child link="${prefix}holder_approach_link"/>
+      <child link="${prefix}holder_approach"/>
     </joint>
-    <link name="${prefix}holder_approach_link"/>
+    <link name="${prefix}holder_approach"/>
+<!--     <joint name="${prefix}grab_joint" type="fixed">
+      <origin rpy="3.1416 0 0" xyz="0 0 0.38"/>
+      <parent link="${prefix}holder_link"/>
+      <child link="${prefix}grab"/>
+    </joint>
+    <link name="${prefix}grab"/> -->
+    <!-- TABLE TAG -->
+    <xacro:ar_tag prefix="${prefix}holder_" parent="${prefix}holder_link" tag_id="${tag_id}">
+      <origin xyz="0 0 0" rpy="0 0 0"/>
+    </xacro:ar_tag>
     <gazebo reference="${prefix}holder_link">
       <visual>

File: component_sorting_description/urdf/table.urdf.xacro (robot description, xacro)
@@ -2,5 +2,5 @@
 <robot name="table" xmlns:xacro="http://wiki.ros.org/xacro">
   <xacro:include filename="$(find component_sorting_description)/urdf/inertia.urdf.xacro" />
-  <xacro:include filename="$(find component_sorting_description)/urdf/box/holder_table.urdf.xacro" />
+  <xacro:include filename="$(find component_sorting_description)/urdf/box/holder.urdf.xacro" />
 <!--   <xacro:include filename="$(find vigir_ar_alvar_description)/urdf/artag.urdf.xacro" /> -->
   <xacro:include filename="$(find component_sorting_description)/ar_tags/ar_tag_12cm_border.urdf.xacro" />
@@ -77,13 +77,13 @@
   <xacro:property name="right_holder_offset_z" value="${table_height/2}"/>
     <!-- HOLDERS -->
-  <xacro:holder_table prefix="${prefix}center_" parent="${prefix}base_link" tag_id="marker2_12cm" >
+  <xacro:holder prefix="${prefix}center_" parent="${prefix}base_link" tag_id="marker2_12cm" >
       <origin xyz="${center_holder_offset_x} ${center_holder_offset_y} ${center_holder_offset_z}" rpy="0 0 0"/>
-  </xacro:holder_table>
-  <xacro:holder_table prefix="${prefix}left_" parent="${prefix}base_link" tag_id="marker3_12cm" >
+  </xacro:holder>
+  <xacro:holder prefix="${prefix}left_" parent="${prefix}base_link" tag_id="marker3_12cm" >
       <origin xyz="${left_holder_offset_x} ${left_holder_offset_y} ${left_holder_offset_z}" rpy="0 0 0"/>
-  </xacro:holder_table>
-  <xacro:holder_table prefix="${prefix}right_" parent="${prefix}base_link" tag_id="marker1_12cm" >
+  </xacro:holder>
+  <xacro:holder prefix="${prefix}right_" parent="${prefix}base_link" tag_id="marker1_12cm" >
       <origin xyz="${right_holder_offset_x} ${right_holder_offset_y} ${right_holder_offset_z}" rpy="0 0 0"/>
-  </xacro:holder_table>
+  </xacro:holder>
   <gazebo reference="${prefix}base_link">
     <material>Gazebo/White</material>
