Commit message: component_sorting_description: updated kairos description

File: component_sorting_description/robots/component_sorting.urdf.xacro (robot description, xacro)
@@ -9,6 +9,7 @@
   	<xacro:arg name="prefix" default="robot_"/>
     <xacro:property name="prefix" value="$(arg prefix)" />
-    <!--xacro:include filename="$(find rbkairos_description)/robots/versions/rbkairos_ur5_oem_vgc10.urdf.xacro" /-->
-    <xacro:include filename="$(find rbkairos_description)/robots/versions/rbkairos_ur5_vgc10.urdf.xacro" />
+    <xacro:property name="PI" value="3.1415926535897931"/>
+    <xacro:include filename="$(find rbkairos_description)/robots/versions/rbkairos_ur5_plus.urdf.xacro" />
+    <!-- <xacro:include filename="$(find rbkairos_description)/robots/versions/rbkairos_ur5_vgc10.urdf.xacro" /> -->
     <!-- Import holder for the boxes -->
 <!-- 	<xacro:include filename="$(find rbkairos_description)/urdf/box/holder.urdf.xacro" /> -->
@@ -19,11 +20,11 @@
     <xacro:property name="center_holder_offset_x" value="-0.2025"/>
     <xacro:property name="center_holder_offset_y" value="0.0"/>
-    <xacro:property name="center_holder_offset_z" value="0.38212"/>
+    <xacro:property name="center_holder_offset_z" value="0.564"/>
     <xacro:property name="left_holder_offset_x" value="-0.2025"/> <!-- -0.195 -->
     <xacro:property name="left_holder_offset_y" value="0.228"/> <!-- 0.225 -->
-    <xacro:property name="left_holder_offset_z" value="0.38212"/>
+    <xacro:property name="left_holder_offset_z" value="0.564"/>
     <xacro:property name="right_holder_offset_x" value="-0.2025"/>
     <xacro:property name="right_holder_offset_y" value="-0.228"/>
-    <xacro:property name="right_holder_offset_z" value="0.38212"/>
+    <xacro:property name="right_holder_offset_z" value="0.564"/>
     <xacro:property name="center_table_holder_offset_x" value="0.68"/>
     <xacro:property name="center_table_holder_offset_y" value="0.0"/>
@@ -36,5 +37,5 @@
     <xacro:property name="right_table_holder_offset_z" value="0.9"/>
     <!-- ROBOT -->
-    <xacro:rbkairos_ur5_oem_vgc10 prefix="$(arg prefix)" publish_bf="true" hq="true" load_kinematics_file="$(arg load_kinematics_file)"/>
+    <xacro:rbkairos prefix="$(arg prefix)" publish_bf="true" hq="true" load_kinematics_file="$(arg load_kinematics_file)"/>
 <!--     <joint name="${prefix}base_boxes" type="fixed">
       <origin rpy="0 0 0" xyz="0 0 0"/>

Commit message: component_sorting_description: add table positions (right, center, left) as static frames

File: component_sorting_description/robots/component_sorting.urdf.xacro (robot description, xacro)
@@ -12,9 +12,16 @@
     <xacro:include filename="$(find component_sorting_description)/robots/rbkairos_ur5_plus.urdf.xacro" />
     <!-- <xacro:include filename="$(find rbkairos_description)/robots/versions/rbkairos_ur5_vgc10.urdf.xacro" /> -->
-    <!-- Import holder for the boxes -->
-<!-- 	<xacro:include filename="$(find rbkairos_description)/urdf/box/holder.urdf.xacro" /> -->
-    <!-- Import  holder for the boxes test -->
-	<xacro:include filename="$(find component_sorting_description)/urdf/box/holder.urdf.xacro" />
-  <xacro:include filename="$(find component_sorting_description)/urdf/inertia.urdf.xacro" />
+    <!-- Import  component sortting application parameters  -->
+    <xacro:property name="objects_config_yaml_file" value="$(find component_sorting)/config/objects_config.yaml" />
+    <xacro:property name="objects_config" value="${load_yaml(objects_config_yaml_file)}"/>
+    <xacro:arg name="table_length" default="0.63"/>
+    <xacro:property name="table_length" value="${objects_config['table']['geometry']['box']['length']}" />
+    <xacro:arg name="table_width" default="0.63"/>
+    <xacro:property name="table_width" value="${objects_config['table']['geometry']['box']['width']}" />
+    <xacro:arg name="table_height" default="0.75"/>
+    <xacro:property name="table_height" value="${objects_config['table']['geometry']['box']['height']}" />
+    <!-- Import  holder  -->
+	  <xacro:include filename="$(find component_sorting_description)/urdf/box/holder.urdf.xacro" />
+    <xacro:include filename="$(find component_sorting_description)/urdf/inertia.urdf.xacro" />
     <!-- Holder parameters -->
     <xacro:property name="center_holder_offset_x" value="-0.2025"/>
@@ -27,13 +34,13 @@
     <xacro:property name="right_holder_offset_y" value="-0.228"/>
     <xacro:property name="right_holder_offset_z" value="0.564"/>
-    <xacro:property name="center_table_holder_offset_x" value="0.68"/>
+    <xacro:property name="center_table_holder_offset_x" value="0.71"/>
     <xacro:property name="center_table_holder_offset_y" value="0.0"/>
-    <xacro:property name="center_table_holder_offset_z" value="0.9"/>
-    <xacro:property name="left_table_holder_offset_x" value="0.68"/>
+    <xacro:property name="center_table_holder_offset_z" value="${table_height}"/>
+    <xacro:property name="left_table_holder_offset_x" value="0.71"/>
     <xacro:property name="left_table_holder_offset_y" value="0.228"/>
-    <xacro:property name="left_table_holder_offset_z" value="0.9"/>
-    <xacro:property name="right_table_holder_offset_x" value="0.68"/>
+    <xacro:property name="left_table_holder_offset_z" value="${table_height}"/>
+    <xacro:property name="right_table_holder_offset_x" value="0.71"/>
     <xacro:property name="right_table_holder_offset_y" value="-0.228"/>
-    <xacro:property name="right_table_holder_offset_z" value="0.9"/>
+    <xacro:property name="right_table_holder_offset_z" value="${table_height}"/>
     <xacro:arg name="ros_planar_move_plugin" default="false"/>
     <!-- ROBOT -->
@@ -42,26 +49,5 @@
       <xacro:omni_steering prefix="$(arg prefix)" publish_tf="true"/>
     </xacro:if>
-<!--     <joint name="${prefix}base_boxes" type="fixed">
-      <origin rpy="0 0 0" xyz="0 0 0"/>
-      <parent link="${prefix}base_chapa"/>
-      <child link="${prefix}base_boxes_link"/>
-    </joint>
-    <link name="${prefix}base_boxes_link">
-      <collision>
-        <origin xyz="0 0 0.0015"/>
-        <geometry>
-          <box size="0.71 0.57 0.003" />
-        </geometry>
-      </collision>
-    </link>
-    <gazebo reference="${prefix}base_boxes_link">
-      <material>Gazebo/White</material>
-      <mu1>1000000.0</mu1>
-      <mu2>1000000.0</mu2>
-      <kp>10000000.0</kp>
-      <kd>1.0</kd>
-      <minDepth>0.001</minDepth>
-    </gazebo> -->
-    <!-- HOLDERS -->
+    <!-- ROBOT HOLDERS -->
      <xacro:holder prefix="${prefix}center_" parent="${prefix}base_link" tag_id="marker5_12cm">
         <origin xyz="${center_holder_offset_x} ${center_holder_offset_y} ${center_holder_offset_z}" rpy="0 0 3.14159"/>
@@ -73,58 +59,47 @@
         <origin xyz="${right_holder_offset_x} ${right_holder_offset_y} ${right_holder_offset_z}" rpy="0 0 3.14159"/>
     </xacro:holder>
-    <!-- BOX -->
-<!--   <joint name="${prefix}joint" type="fixed">
-    <origin rpy="0 0 0" xyz="0 0 0.01"/>
-    <parent link="${prefix}right_table_holder_link"/>
-    <child link="${prefix}body_box_link"/>
-  </joint>
-  <link name="${prefix}body_box_link">
-    <inertial>
-      <mass value="5" />
-      <origin xyz="0 0 0.05" />
-      <solid_cuboid_inertia m="5" h="0.2" d="0.1" w="0.3"/>
-    </inertial>
-    <visual>
-      <origin rpy="0 0 0" xyz="0 0 0"/>
-      <geometry>
-        <mesh filename="package://component_sorting_description/meshes/box/box_base.stl"/>
-      </geometry>
-    </visual>
-    <collision>
-      <origin rpy="0 0 0" xyz="0 0 0"/>
-      <geometry>
-        <mesh filename="package://component_sorting_description/meshes/box/box_base.stl"/>
-      </geometry>
-    </collision>
-  </link>
-  <joint name="${prefix}handle_joint" type="fixed">
-    <origin rpy="0 0 0" xyz="0 0 0.1"/>
-    <parent link="${prefix}body_box_link"/>
-    <child link="${prefix}handle_link"/>
-  </joint>
-  <link name="${prefix}handle_link">
-    <inertial>
-      <mass value="0.1" />
-      <origin xyz="0 0 0" />
-      <solid_cuboid_inertia m="0.1" h="0.2" d="0.01" w="0.3"/>
-    </inertial>
-    <visual>
-      <origin rpy="0 0 0" xyz="0 0 0"/>
-      <geometry>
-        <mesh filename="package://component_sorting_description/meshes/box/handle.stl"/>
-      </geometry>
-    </visual>
-    <collision>
-      <origin rpy="0 0 0" xyz="0 0 0"/>
-      <geometry>
-        <mesh filename="package://component_sorting_description/meshes/box/handle.stl"/>
-      </geometry>
-    </collision>
-  </link>
-  <joint name="${prefix}grasping_joint" type="fixed">
-    <origin rpy="3.141592 0 0" xyz="0 0 0.25"/>
-    <parent link="${prefix}body_box_link"/>
-    <child link="${prefix}grasping_link"/>
-  </joint>
-  <link name="${prefix}grasping_link"/> -->
+    <!--TABLE HOLDER STATIC POSITIONS -->
+    <joint name="table_center_holder_joint" type="fixed">
+      <origin rpy="0 0 0" xyz="${center_table_holder_offset_x} ${center_table_holder_offset_y} ${center_table_holder_offset_z}"/>
+      <parent link="${prefix}base_footprint"/>
+      <child link="table_center_holder_link"/>
+    </joint>
+    <link name="table_center_holder_link">
+    </link>
+    <joint name="table_right_holder_joint" type="fixed">
+      <origin rpy="0 0 0" xyz="${right_table_holder_offset_x} ${right_table_holder_offset_y} ${right_table_holder_offset_z}"/>
+      <parent link="${prefix}base_footprint"/>
+      <child link="table_right_holder_link"/>
+    </joint>
+    <link name="table_right_holder_link">
+    </link>
+    <joint name="table_left_holder_joint" type="fixed">
+      <origin rpy="0 0 0" xyz="${left_table_holder_offset_x} ${left_table_holder_offset_y} ${left_table_holder_offset_z}"/>
+      <parent link="${prefix}base_footprint"/>
+      <child link="table_left_holder_link"/>
+    </joint>
+    <link name="table_left_holder_link">
+    </link>
+    <!--TABLE HOLDER ORIENTED STATIC POSITIONS -->
+    <joint name="table_center_holder_oriented_joint" type="fixed">
+      <origin rpy="${-3.14159} 0 ${-3.14159/2}" xyz="${center_table_holder_offset_x} ${center_table_holder_offset_y} ${center_table_holder_offset_z}"/>
+      <parent link="${prefix}base_footprint"/>
+      <child link="table_center_holder_oriented_link"/>
+    </joint>
+    <link name="table_center_holder_oriented_link">
+    </link>
+    <joint name="table_right_holder_oriented_joint" type="fixed">
+      <origin rpy="${-3.14159} 0 ${-3.14159/2}" xyz="${right_table_holder_offset_x} ${right_table_holder_offset_y} ${right_table_holder_offset_z}"/>
+      <parent link="${prefix}base_footprint"/>
+      <child link="table_right_holder_oriented_link"/>
+    </joint>
+    <link name="table_right_holder_oriented_link">
+    </link>
+    <joint name="table_left_holder_oriented_joint" type="fixed">
+      <origin rpy="${-3.14159} 0 ${-3.14159/2}" xyz="${left_table_holder_offset_x} ${left_table_holder_offset_y} ${left_table_holder_offset_z}"/>
+      <parent link="${prefix}base_footprint"/>
+      <child link="table_left_holder_oriented_link"/>
+    </joint>
+    <link name="table_left_holder_oriented_link">
+    </link>
 </robot>
