Commit message: component_sorting_description: remove unecessary meshes and urdf files (hr-recycler holders and boxes)

File: component_sorting_description/robots/component_sorting.urdf.xacro (robot description, xacro)
@@ -11,36 +11,5 @@
     <xacro:property name="PI" value="3.1415926535897931"/>
     <xacro:include filename="$(find component_sorting_description)/robots/rbkairos_ur5_plus.urdf.xacro" />
-    <!-- <xacro:include filename="$(find rbkairos_description)/robots/versions/rbkairos_ur5_vgc10.urdf.xacro" /> -->
-    <!-- Import  component sortting application parameters  -->
-    <xacro:property name="objects_config_yaml_file" value="$(find component_sorting)/config/objects_config.yaml" />
-    <xacro:property name="objects_config" value="${load_yaml(objects_config_yaml_file)}"/>
-    <xacro:arg name="table_length" default="0.63"/>
-    <xacro:property name="table_length" value="${objects_config['table']['geometry']['box']['length']}" />
-    <xacro:arg name="table_width" default="0.63"/>
-    <xacro:property name="table_width" value="${objects_config['table']['geometry']['box']['width']}" />
-    <xacro:arg name="table_height" default="0.75"/>
-    <xacro:property name="table_height" value="${objects_config['table']['geometry']['box']['height']}" />
-    <!-- Import  holder  -->
-	  <xacro:include filename="$(find component_sorting_description)/urdf/box/holder.urdf.xacro" />
     <xacro:include filename="$(find component_sorting_description)/urdf/inertia.urdf.xacro" />
-    <!-- Holder parameters -->
-    <xacro:property name="center_holder_offset_x" value="-0.2025"/>
-    <xacro:property name="center_holder_offset_y" value="0.0"/>
-    <xacro:property name="center_holder_offset_z" value="0.564"/>
-    <xacro:property name="left_holder_offset_x" value="-0.2025"/> <!-- -0.195 -->
-    <xacro:property name="left_holder_offset_y" value="0.228"/> <!-- 0.225 -->
-    <xacro:property name="left_holder_offset_z" value="0.564"/>
-    <xacro:property name="right_holder_offset_x" value="-0.2025"/>
-    <xacro:property name="right_holder_offset_y" value="-0.228"/>
-    <xacro:property name="right_holder_offset_z" value="0.564"/>
-    <xacro:property name="center_table_holder_offset_x" value="0.71"/>
-    <xacro:property name="center_table_holder_offset_y" value="0.0"/>
-    <xacro:property name="center_table_holder_offset_z" value="${table_height}"/>
-    <xacro:property name="left_table_holder_offset_x" value="0.71"/>
-    <xacro:property name="left_table_holder_offset_y" value="0.228"/>
-    <xacro:property name="left_table_holder_offset_z" value="${table_height}"/>
-    <xacro:property name="right_table_holder_offset_x" value="0.71"/>
-    <xacro:property name="right_table_holder_offset_y" value="-0.228"/>
-    <xacro:property name="right_table_holder_offset_z" value="${table_height}"/>
     <xacro:arg name="ros_planar_move_plugin" default="false"/>
     <!-- ROBOT -->
@@ -49,57 +18,3 @@
       <xacro:omni_steering prefix="$(arg prefix)" publish_tf="true"/>
     </xacro:if>
-    <!-- ROBOT HOLDERS -->
-     <xacro:holder prefix="${prefix}center_" parent="${prefix}base_link" tag_id="marker5_12cm">
-        <origin xyz="${center_holder_offset_x} ${center_holder_offset_y} ${center_holder_offset_z}" rpy="0 0 3.14159"/>
-    </xacro:holder>
-    <xacro:holder prefix="${prefix}left_" parent="${prefix}base_link" tag_id="marker6_12cm">
-        <origin xyz="${left_holder_offset_x} ${left_holder_offset_y} ${left_holder_offset_z}" rpy="0 0 3.14159"/>
-    </xacro:holder>
-    <xacro:holder prefix="${prefix}right_" parent="${prefix}base_link" tag_id="marker4_12cm" >
-        <origin xyz="${right_holder_offset_x} ${right_holder_offset_y} ${right_holder_offset_z}" rpy="0 0 3.14159"/>
-    </xacro:holder>
-    <!--TABLE HOLDER STATIC POSITIONS -->
-    <joint name="table_center_holder_joint" type="fixed">
-      <origin rpy="0 0 0" xyz="${center_table_holder_offset_x} ${center_table_holder_offset_y} ${center_table_holder_offset_z}"/>
-      <parent link="${prefix}base_footprint"/>
-      <child link="table_center_holder_link"/>
-    </joint>
-    <link name="table_center_holder_link">
-    </link>
-    <joint name="table_right_holder_joint" type="fixed">
-      <origin rpy="0 0 0" xyz="${right_table_holder_offset_x} ${right_table_holder_offset_y} ${right_table_holder_offset_z}"/>
-      <parent link="${prefix}base_footprint"/>
-      <child link="table_right_holder_link"/>
-    </joint>
-    <link name="table_right_holder_link">
-    </link>
-    <joint name="table_left_holder_joint" type="fixed">
-      <origin rpy="0 0 0" xyz="${left_table_holder_offset_x} ${left_table_holder_offset_y} ${left_table_holder_offset_z}"/>
-      <parent link="${prefix}base_footprint"/>
-      <child link="table_left_holder_link"/>
-    </joint>
-    <link name="table_left_holder_link">
-    </link>
-    <!--TABLE HOLDER ORIENTED STATIC POSITIONS -->
-    <joint name="table_center_holder_oriented_joint" type="fixed">
-      <origin rpy="${-3.14159} 0 ${-3.14159/2}" xyz="${center_table_holder_offset_x} ${center_table_holder_offset_y} ${center_table_holder_offset_z}"/>
-      <parent link="${prefix}base_footprint"/>
-      <child link="table_center_holder_oriented_link"/>
-    </joint>
-    <link name="table_center_holder_oriented_link">
-    </link>
-    <joint name="table_right_holder_oriented_joint" type="fixed">
-      <origin rpy="${-3.14159} 0 ${-3.14159/2}" xyz="${right_table_holder_offset_x} ${right_table_holder_offset_y} ${right_table_holder_offset_z}"/>
-      <parent link="${prefix}base_footprint"/>
-      <child link="table_right_holder_oriented_link"/>
-    </joint>
-    <link name="table_right_holder_oriented_link">
-    </link>
-    <joint name="table_left_holder_oriented_joint" type="fixed">
-      <origin rpy="${-3.14159} 0 ${-3.14159/2}" xyz="${left_table_holder_offset_x} ${left_table_holder_offset_y} ${left_table_holder_offset_z}"/>
-      <parent link="${prefix}base_footprint"/>
-      <child link="table_left_holder_oriented_link"/>
-    </joint>
-    <link name="table_left_holder_oriented_link">
-    </link>
 </robot>

File: component_sorting_description/robots/rbkairos_ur5_plus.urdf.xacro (robot description, xacro)
@@ -177,34 +177,4 @@
           <!--<origin xyz="0.07 0.0 0.065" rpy="${pi} ${-pi/2} 0"/>-->
     <!--</xacro:sensor_intel_d435>-->
-    <gazebo>
-      <plugin name="ground_truth_controller" filename="librobotnik_gazebo_ground_truth_odom.so">
-        <alwaysOn>true</alwaysOn>
-        <updateRate>50.0</updateRate>
-        <bodyName>${prefix}base_link</bodyName> <!-- robot body to track, in gazebo -->
-        <frameName>base_link_gt</frameName> <!-- frame name of robot body to be published in ros -->
-        <worldBodyName>world</worldBodyName> <!-- fixed body where body is tracked, in gazebo -->
-        <worldFrameName>odom</worldFrameName> <!-- frame name of fixed body to be published in ros -->
-        <topicName>odom_gt</topicName>
-        <gaussianNoise>0.01</gaussianNoise>
-        <xyzOffsets>0 0 0</xyzOffsets>
-        <rpyOffsets>0 0 0</rpyOffsets>
-        <broadcastTF>True</broadcastTF>
-      </plugin>
-    </gazebo>
-    <gazebo>
-      <plugin name="ground_lasertruth_controller_" filename="librobotnik_gazebo_ground_truth_odom.so">
-        <alwaysOn>true</alwaysOn>
-        <updateRate>50.0</updateRate>
-        <bodyName>${prefix}front_laser_link</bodyName> <!-- robot body to track, in gazebo -->
-        <frameName>laser_gt</frameName> <!-- frame name of robot body to be published in ros -->
-        <worldBodyName>world</worldBodyName> <!-- fixed body where body is tracked, in gazebo -->
-        <worldFrameName>odom</worldFrameName> <!-- frame name of fixed body to be published in ros -->
-        <topicName>laser_gt</topicName>
-        <gaussianNoise>0.01</gaussianNoise>
-        <xyzOffsets>0 0 0</xyzOffsets>
-        <rpyOffsets>0 0 0</rpyOffsets>
-        <broadcastTF>True</broadcastTF>
-      </plugin>
-    </gazebo>
   </xacro:macro>
   <!-- Gazebo ros control pluggins -->

File: component_sorting_description/urdf/package.urdf.xacro (robot description, xacro)
@@ -10,5 +10,5 @@
   </link>
   <joint name="${prefix}joint" type="fixed">
-    <origin rpy="0 0 0" xyz="0 0 0"/>
+    <origin rpy="0 0 -1.5708" xyz="0 0 0"/>
     <parent link="${prefix}base_link"/>
     <child link="${prefix}body_box_link"/>
@@ -21,13 +21,13 @@
     </inertial>
     <visual>
-      <origin rpy="0 0 0" xyz="0 0 0"/>
+      <origin rpy="0 0 0" xyz="0 0 0.05"/>
       <geometry>
-        <mesh filename="package://component_sorting_description/meshes/box/box_base.stl"/>
+        <box size="0.15 0.25 0.10" />
       </geometry>
     </visual>
     <collision>
-      <origin rpy="0 0 0" xyz="0 0 0"/>
+      <origin rpy="0 0 0" xyz="0 0 0.05"/>
       <geometry>
-        <mesh filename="package://component_sorting_description/meshes/box/box_base.stl"/>
+        <box size="0.15 0.25 0.10" />
       </geometry>
 <surface>
@@ -53,39 +53,13 @@
     </collision>
   </link>
-  <joint name="${prefix}handle_joint" type="prismatic">
-    <axis xyz="0 0 1"/>
-    <limit effort="1000.0" lower="-0.02" upper="0.02" velocity="0.5"/>
-    <origin rpy="0 0 0" xyz="0 0 0.1"/>
+  <joint name="${prefix}qr_joint" type="fixed">
+    <origin rpy="0 0 0" xyz="0 0 0.05"/>
     <parent link="${prefix}body_box_link"/>
-    <child link="${prefix}handle_link"/>
+    <child link="${prefix}qr"/>
   </joint>
-  <link name="${prefix}handle_link">
-    <inertial>
-      <mass value="0.1" />
-      <origin xyz="0 0 0" />
-      <solid_cuboid_inertia m="0.1" h="0.2" d="0.01" w="0.3"/>
-    </inertial>
-    <visual>
-      <origin rpy="0 0 0" xyz="0 0 0"/>
-      <geometry>
-        <mesh filename="package://component_sorting_description/meshes/box/handle.stl"/>
-      </geometry>
-    </visual>
-    <collision>
-      <origin rpy="0 0 0" xyz="0 0 0"/>
-      <geometry>
-        <mesh filename="package://component_sorting_description/meshes/box/handle.stl"/>
-      </geometry>
-    </collision>
-  </link>
-  <joint name="${prefix}grasping_joint" type="fixed">
-    <origin rpy="3.141592 0 0" xyz="0 0 0.158"/>
-    <parent link="${prefix}handle_link"/>
-    <child link="${prefix}grasping_link"/>
-  </joint>
-  <link name="${prefix}grasping_link"/>
+  <link name="${prefix}qr"/>
   <!-- AR TAG -->
-  <xacro:ar_tag prefix="${prefix}" parent="${prefix}handle_link" tag_id="${tag_id}">
-    <origin xyz="0 0 0.1575" rpy="0 0 ${-3.14159/2}"/>
+  <xacro:ar_tag prefix="${prefix}" parent="${prefix}qr" tag_id="${tag_id}">
+    <origin xyz="0 0 0.05" rpy="0 0 0"/>
   </xacro:ar_tag>
 <!--  <xacro:artag name="artag_01" parent="${prefix}grasping_link">
@@ -109,13 +83,3 @@
     <maxContacts>10</maxContacts>
  </gazebo>
-  <gazebo reference="${prefix}handle_link">
-    <visual>
-      <material>
-        <ambient>0.0 0.0 0.0 1.0</ambient>
-        <diffuse>0.2 0.2 0.2 1.0</diffuse>
-        <specular>0.584313725 0.647058824 0.650980392 1.0</specular>
-        <emissive>0.0 0.0 0.0 0.0</emissive>
-      </material>
-    </visual>
-  </gazebo>
 </robot>

File: component_sorting_description/urdf/table.urdf.xacro (robot description, xacro)
@@ -7,8 +7,6 @@
   <xacro:arg name="prefix" default="table_"/>
   <xacro:property name="prefix" value="$(arg prefix)" />
-  <xacro:property name="objects_config_yaml_file" value="$(find component_sorting)/config/objects_config.yaml" />
+  <xacro:property name="objects_config_yaml_file" value="$(find component_sorting_description)/config/layout.yaml" />
   <xacro:property name="objects_config" value="${load_yaml(objects_config_yaml_file)}"/>
-  <xacro:property name="component_sorting_yaml_file" value="$(find component_sorting)/config/component_sorting.yaml" />
-  <xacro:property name="component_sorting" value="${load_yaml(component_sorting_yaml_file)}"/>
   <xacro:arg name="table_length" default="0.63"/>
   <xacro:property name="table_length" value="${objects_config['table']['geometry']['box']['length']}" />
@@ -17,8 +15,4 @@
   <xacro:arg name="table_height" default="0.75"/>
   <xacro:property name="table_height" value="${objects_config['table']['geometry']['box']['height']}" />
-  <xacro:arg name="holder_width" default="0.228"/>
-  <xacro:property name="holder_width" value="${component_sorting['holder']['width']}" />
-  <xacro:arg name="holder_length" default="0.30"/>
-  <xacro:property name="holder_length" value="${component_sorting['holder']['length']}" />
   <xacro:arg name="qr_height" default="0.375"/>
   <xacro:property name="qr_height" value="${objects_config['table']['geometry']['qr']['height']}" />
@@ -84,14 +78,4 @@
   <xacro:property name="right_holder_offset_y" value="${-holder_width}"/>
   <xacro:property name="right_holder_offset_z" value="${table_height}"/>
-    <!-- HOLDERS -->
-<!--   <xacro:holder prefix="${prefix}center_" parent="${prefix}base_link" tag_id="marker2_12cm" >
-      <origin xyz="${center_holder_offset_x} ${center_holder_offset_y} ${center_holder_offset_z}" rpy="0 0 0"/>
-  </xacro:holder>
-  <xacro:holder prefix="${prefix}left_" parent="${prefix}base_link" tag_id="marker3_12cm" >
-      <origin xyz="${left_holder_offset_x} ${left_holder_offset_y} ${left_holder_offset_z}" rpy="0 0 0"/>
-  </xacro:holder>
-  <xacro:holder prefix="${prefix}right_" parent="${prefix}base_link" tag_id="marker1_12cm" >
-      <origin xyz="${right_holder_offset_x} ${right_holder_offset_y} ${right_holder_offset_z}" rpy="0 0 0"/>
-  </xacro:holder> -->
   <gazebo reference="${prefix}base_link">
     <material>Gazebo/White</material>
