Commit message: component_sorting_description: - added ur5e joint limit configuration yaml (joint limited configuration) - updated urdf component sorting with correct ur arm and orientation - removed collision in holders

File: component_sorting_description/robots/rbkairos_ur5_plus.urdf.xacro (robot description, xacro)
@@ -8,5 +8,5 @@
   <xacro:include filename="$(find summit_xl_description)/urdf/bases/summit_xlsk_base_plus.urdf.xacro" />
   <!-- Include UR-5 ARM -->
-  <xacro:include filename="$(find ur_description)/urdf/inc/ur5_macro.xacro" />
+  <xacro:include filename="$(find ur_description)/urdf/inc/ur5e_macro.xacro" />
   <!-- Include OnRobot vgc10 -->
   <xacro:include filename="$(find rbkairos_description)/urdf/structures/vgc10.urdf.xacro" />
@@ -32,5 +32,5 @@
   <xacro:property name="arm_orientation_r" value="0"/>
   <xacro:property name="arm_orientation_p" value="0"/>
-  <xacro:property name="arm_orientation_y" value="0"/>
+  <xacro:property name="arm_orientation_y" value="${PI}"/>
   <!-- Wheel parameters -->
   <xacro:property name="wheel_offset_x" value="0.21528" />    <!-- x,y,z in translation from base_link to the center of the wheel -->
@@ -57,5 +57,5 @@
   <xacro:property name="front_rgbd_camera_offset_z" value="0.25062"/>
   <xacro:property name="arm_rgbd_camera_offset_x" value="0.0"/>
-  <xacro:property name="arm_rgbd_camera_offset_y" value="0.0876"/>
+  <xacro:property name="arm_rgbd_camera_offset_y" value="-0.0876"/>
   <xacro:property name="arm_rgbd_camera_offset_z" value="0.0475"/>
   <xacro:property name="gps_offset_x" value="-0.365"/>
@@ -83,5 +83,5 @@
   <xacro:property name="arm_orientation_r" value="0"/>
   <xacro:property name="arm_orientation_p" value="0"/>
-  <xacro:property name="arm_orientation_y" value="0"/>
+  <xacro:property name="arm_orientation_y" value="${PI}"/>
   <xacro:macro name="rbkairos" params="prefix publish_bf hq load_kinematics_file gpu:=false">
     <!-- *************** -->
@@ -104,6 +104,6 @@
     </xacro:omni_wheel>
     <!-- UR-5 ARM -->
-    <xacro:ur5_robot prefix="$(arg prefix)arm_" >
-    </xacro:ur5_robot>
+    <xacro:ur5e_robot prefix="$(arg prefix)arm_" joint_limits_parameters_file='$(find component_sorting_description)/config/joint_limits.yaml'>
+    </xacro:ur5e_robot>
     <joint name="${prefix}arm_base_joint" type="fixed">
       <origin xyz="${arm_position_x} ${arm_position_y} ${arm_position_z}" rpy="${arm_orientation_r} ${arm_orientation_p} ${arm_orientation_y}"/>
@@ -113,5 +113,5 @@
     <!-- OnRobot VGC-10 -->
     <xacro:vgc10 prefix="${prefix}vgc10" parent="${prefix}arm_tool0">
-        <origin xyz="0 0 0.01" rpy="0 -${PI/2.0} ${PI}"/>
+        <origin xyz="0 0 0.01" rpy="0 -${PI/2.0} ${PI/2}"/>
     </xacro:vgc10>
     <!-- IMU -->
@@ -130,8 +130,8 @@
     </xacro:sensor_intel_d435>
     <xacro:sensor_orbbec_astra_embedded_s prefix="${prefix}arm_rgbd_camera" parent="${prefix}arm_tool0" prefix_topic="arm_rgbd_camera">
-      <origin xyz="${arm_rgbd_camera_offset_x} ${arm_rgbd_camera_offset_y} ${arm_rgbd_camera_offset_z}" rpy="0 ${-PI/2} ${-PI/2}"/>
+      <origin xyz="${arm_rgbd_camera_offset_x} ${arm_rgbd_camera_offset_y} ${arm_rgbd_camera_offset_z}" rpy="0 ${-PI/2} ${PI/2}"/>
     </xacro:sensor_orbbec_astra_embedded_s>
     <joint name="$(arg prefix)arm_camera_support" type="fixed">
-      <origin xyz="0 0 0" rpy="0 0 0"/>
+      <origin xyz="0 0 0" rpy="0 0 ${PI}"/>
       <parent link="$(arg prefix)arm_tool0" />
       <child link="$(arg prefix)arm_camera_support_link" />
@@ -140,9 +140,9 @@
       <inertial>
         <mass value="0.2" />
-        <origin xyz="0 0 0" />
+        <origin rpy="0 -${PI/2.0} -${PI/2.0}" xyz="-0.038 -0.038 0"/>
         <solid_cuboid_inertia m="0.2" h="0.015" d="0.05" w="0.015"/>
       </inertial>
       <visual>
-        <origin rpy="0 -${PI/2.0} -${PI/2.0}" xyz="-0.035 -0.035 0"/>
+        <origin rpy="0 -${PI/2.0} -${PI/2.0}" xyz="-0.038 -0.038 0"/>
         <geometry>
           <mesh filename="package://component_sorting_description/meshes/embedded_s_support.dae"/>
@@ -150,5 +150,5 @@
       </visual>
       <collision>
-        <origin rpy="0 -${PI/2.0} -${PI/2.0}" xyz="-0.035 -0.035 0"/>
+        <origin rpy="0 -${PI/2.0} -${PI/2.0}" xyz="-0.038 -0.038 0"/>
         <geometry>
           <mesh filename="package://component_sorting_description/meshes/embedded_s_support.dae"/>

File: component_sorting_description/urdf/box/holder.urdf.xacro (robot description, xacro)
@@ -31,23 +31,30 @@
         </geometry>
       </visual>
-      <collision>
+      <!--collision>
         <origin rpy="0 0 0" xyz="0 0 0"/>
         <geometry>
           <mesh filename="package://component_sorting_description/meshes/box/box_holder.stl"/>
         </geometry>
-      </collision>
+      </collision-->
+    </link>
+    <joint name="${prefix}holder_oriented_joint" type="fixed">
+      <origin rpy="${-3.14159} 0 ${-3.14159/2}" xyz="0 0 0"/>
+      <parent link="${prefix}holder_link"/>
+      <child link="${prefix}holder_oriented_link"/>
+    </joint>
+    <link name="${prefix}holder_oriented_link">
     </link>
     <joint name="${prefix}holder_approach_joint" type="fixed">
-      <origin rpy="3.1416 0 0" xyz="-0.137 0 0.50"/>
-      <parent link="${prefix}holder_link"/>
+      <origin rpy="0 0 0" xyz="0 0.137 -0.50"/>
+      <parent link="${prefix}holder_oriented_link"/>
       <child link="${prefix}holder_approach"/>
     </joint>
     <link name="${prefix}holder_approach"/>
-<!--     <joint name="${prefix}grab_joint" type="fixed">
-      <origin rpy="3.1416 0 0" xyz="0 0 0.38"/>
-      <parent link="${prefix}holder_link"/>
-      <child link="${prefix}grab"/>
+    <joint name="${prefix}grab_joint" type="fixed">
+      <origin rpy="0 0 0" xyz="0 0 -0.5"/>
+      <parent link="${prefix}holder_oriented_link"/>
+      <child link="${prefix}grab_link"/>
     </joint>
-    <link name="${prefix}grab"/> -->
+    <link name="${prefix}grab_link"/>
     <!-- TABLE TAG -->
     <xacro:ar_tag prefix="${prefix}holder_" parent="${prefix}holder_link" tag_id="${tag_id}">

Commit message: component_sorting_description: update robot description

File: component_sorting_description/robots/rbkairos_ur5_plus.urdf.xacro (robot description, xacro)
@@ -57,6 +57,6 @@
   <xacro:property name="front_rgbd_camera_offset_z" value="0.25062"/>
   <xacro:property name="arm_rgbd_camera_offset_x" value="0.0"/>
-  <xacro:property name="arm_rgbd_camera_offset_y" value="-0.0876"/>
-  <xacro:property name="arm_rgbd_camera_offset_z" value="0.0475"/>
+  <xacro:property name="arm_rgbd_camera_offset_y" value="-0.095"/>
+  <xacro:property name="arm_rgbd_camera_offset_z" value="0.075"/>
   <xacro:property name="gps_offset_x" value="-0.365"/>
   <xacro:property name="gps_offset_y" value="-0.167"/>
@@ -129,6 +129,12 @@
       <origin xyz="${front_rgbd_camera_offset_x} ${front_rgbd_camera_offset_y} ${front_rgbd_camera_offset_z}" rpy="0 0 0"/>
     </xacro:sensor_intel_d435>
-    <xacro:sensor_orbbec_astra_embedded_s prefix="${prefix}arm_rgbd_camera" parent="${prefix}arm_tool0" prefix_topic="arm_rgbd_camera">
+    <joint name="$(arg prefix)small_camera_rotation" type="fixed">
       <origin xyz="${arm_rgbd_camera_offset_x} ${arm_rgbd_camera_offset_y} ${arm_rgbd_camera_offset_z}" rpy="0 ${-PI/2} ${PI/2}"/>
+      <parent link="$(arg prefix)arm_tool0" />
+      <child link="$(arg prefix)rotated_arm_camera" />
+    </joint>
+    <link name="$(arg prefix)rotated_arm_camera"/>
+    <xacro:sensor_orbbec_astra_embedded_s prefix="${prefix}arm_camera" parent="${prefix}rotated_arm_camera" prefix_topic="arm_rgbd_camera">
+      <origin xyz="0 -0.02 0.01" rpy="0 0 ${2*PI/180}"/>
     </xacro:sensor_orbbec_astra_embedded_s>
     <joint name="$(arg prefix)arm_camera_support" type="fixed">

File: component_sorting_description/urdf/box/holder.urdf.xacro (robot description, xacro)
@@ -52,5 +52,5 @@
     <link name="${prefix}holder_approach"/>
     <joint name="${prefix}grab_joint" type="fixed">
-      <origin rpy="0 0 0" xyz="0 0 -0.236"/>
+      <origin rpy="0 0 0" xyz="0 0 -0.23"/>
       <parent link="${prefix}holder_oriented_link"/>
       <child link="${prefix}grab_link"/>

Commit message: modified rbkairos urdf to include the vacuum gripper adapter

File: component_sorting_description/robots/rbkairos_ur5_plus.urdf.xacro (robot description, xacro)
@@ -11,4 +11,5 @@
   <!-- Include OnRobot vgc10 -->
   <xacro:include filename="$(find rbkairos_description)/urdf/structures/vgc10.urdf.xacro" />
+  <xacro:include filename="$(find rbkairos_description)/urdf/structures/vgc10_with_reamer.urdf.xacro" />
   <xacro:include filename="$(find rbkairos_description)/urdf/structures/vgc10.gazebo.xacro" />
   <xacro:include filename="$(find rbkairos_description)/urdf/structures/realsense2vgc10_support.urdf.xacro" />
@@ -111,8 +112,12 @@
       <child link="${prefix}arm_base_link" />
     </joint>
-    <!-- OnRobot VGC-10 -->
-    <xacro:vgc10 prefix="${prefix}vgc10" parent="${prefix}arm_tool0">
+    <!-- OnRobot VGC-10               Task: COMPONENT SORTING -->
+    <!--xacro:vgc10 prefix="${prefix}vgc10" parent="${prefix}arm_tool0">
         <origin xyz="0 0 0.01" rpy="0 -${PI/2.0} ${PI/2}"/>
-    </xacro:vgc10>
+    </xacro:vgc10-->
+    <!-- OnRobot VGC-10 with reamer   Task: DISASSEMBLY       -->
+    <xacro:vgc10_with_reamer prefix="${prefix}vgc10" parent="${prefix}arm_tool0">
+        <origin xyz="0 0 0" rpy="0 0 ${-M_PI/2}"/>
+    </xacro:vgc10_with_reamer>
     <!-- IMU -->
     <xacro:sensor_imu_hector prefix="${prefix}imu" parent="${prefix}base_link">
